File: TSAL/TSAL/TSAL.sch (KiCad schematic (older format))
At the start: 10 parts

Commit message: finished TSAL rev1
Parts:
- removed U?: LTV-817, Package_DIP:DIP-4_W7.62mm, symbol Isolator:LTV-817
- added H1: M3, MountingHole:MountingHole_3.2mm_M3, symbol Mechanical:MountingHole
- added J1, J2, J4: Conn_01x02, Connector_TE-Connectivity:TE_MATE-N-LOK_1-770866-x_1x02_P4.14mm_Vertical, symbol Connector_Generic:Conn_01x02
- added R1: 39k, Resistor_THT:R_Axial_DIN0617_L17.0mm_D6.0mm_P30.48mm_Horizontal, symbol Device:R
- added U1: LTV-817S, Package_DIP:SMDIP-4_W9.53mm, symbol Isolator:LTV-817S
- C1, C2: renamed from C?; footprint (none) -> Capacitor_SMD:C_0603_1608Metric_Pad1.05x0.95mm_HandSolder
- J3: renamed from J?; footprint (none) -> Connector_TE-Connectivity:TE_MATE-N-LOK_1-770866-x_1x02_P4.14mm_Vertical
- Q1: renamed from Q?; footprint (none) -> Package_TO_SOT_SMD:TO-252-3_TabPin2
- R2, R5: renamed from R?; footprint (none) -> Resistor_SMD:R_0603_1608Metric_Pad1.05x0.95mm_HandSolder
- R3: renamed from R?; value R -> 100k; footprint (none) -> Resistor_SMD:R_0603_1608Metric_Pad1.05x0.95mm_HandSolder
- R4: renamed from R?; value R -> 235k; footprint (none) -> Resistor_SMD:R_0603_1608Metric_Pad1.05x0.95mm_HandSolder
- gave numbers to parts that had none: 1
Connections:
- net labels added: HV+, HV-
- wire segments 29 -> 37
Other:
- note added: "High Voltage"
Changed lines of the file:
@@
 $EndDescr
 $Comp
-L Timer:LM555xM U?
+L Timer:LM555xM U2
 U 1 1 5F9882FA
 P 5225 3150
-F 0 "U?" H 5225 3100 50  0000 C CNN
+F 0 "U2" H 5225 3100 50  0000 C CNN
 F 1 "LM555xM" H 5225 3200 50  0000 C CNN
 F 2 "Package_SO:SOIC-8_3.9x4.9mm_P1.27mm" H 6075 2750 50  0001 C CNN
@@
 $EndComp
 $Comp
-L power:GND #PWR?
+L power:GND #PWR0101
 U 1 1 5F989169
 P 5225 4025
-F 0 "#PWR?" H 5225 3775 50  0001 C CNN
+F 0 "#PWR0101" H 5225 3775 50  0001 C CNN
 F 1 "GND" H 5230 3852 50  0000 C CNN
 F 2 "" H 5225 4025 50  0001 C CNN
@@
 	5225 2450 5225 2750
 $Comp
-L Device:R R?
+L Device:R R5
 U 1 1 5F98E1B6
 P 7175 3050
-F 0 "R?" V 7075 3050 50  0000 C CNN
+F 0 "R5" V 7075 3050 50  0000 C CNN
 F 1 "10k" V 7175 3050 50  0000 C CNN
-F 2 "" V 7105 3050 50  0001 C CNN
+F 2 "Resistor_SMD:R_0603_1608Metric_Pad1.05x0.95mm_HandSolder" V 7105 3050 50  0001 C CNN
 F 3 "~" H 7175 3050 50  0001 C CNN
 	1    7175 3050
@@
 $EndComp
 $Comp
-L Device:Q_NMOS_GDS Q?
+L Device:Q_NMOS_GDS Q1
 U 1 1 5F98B2DE
 P 7725 3050
-F 0 "Q?" H 7929 3096 50  0000 L CNN
+F 0 "Q1" H 7929 3096 50  0000 L CNN
 F 1 "Q_NMOS_GDS" H 7929 3005 50  0000 L CNN
-F 2 "" H 7925 3150 50  0001 C CNN
+F 2 "Package_TO_SOT_SMD:TO-252-3_TabPin2" H 7925 3150 50  0001 C CNN
 F 3 "~" H 7725 3050 50  0001 C CNN
 	1    7725 3050
@@
 $EndComp
 $Comp
-L power:GND #PWR?
+L power:GND #PWR0102
 U 1 1 5F98F10A
 P 7825 3250
-F 0 "#PWR?" H 7825 3000 50  0001 C CNN
+F 0 "#PWR0102" H 7825 3000 50  0001 C CNN
 F 1 "GND" H 7830 3077 50  0000 C CNN
 F 2 "" H 7825 3250 50  0001 C CNN
@@
 	7825 2725 7825 2850
 $Comp
-L Connector_Generic:Conn_01x02 J?
+L Connector_Generic:Conn_01x02 J3
 U 1 1 5F996B98
 P 8775 2725
-F 0 "J?" H 8855 2717 50  0000 L CNN
+F 0 "J3" H 8855 2717 50  0000 L CNN
 F 1 "Conn_01x02" H 8855 2626 50  0000 L CNN
-F 2 "" H 8775 2725 50  0001 C CNN
+F 2 "Connector_TE-Connectivity:TE_MATE-N-LOK_1-770866-x_1x02_P4.14mm_Vertical" H 8775 2725 50  0001 C CNN
 F 3 "~" H 8775 2725 50  0001 C CNN
 	1    8775 2725
@@
 $EndComp
 $Comp
-L power:GND #PWR?
+L power:GND #PWR0103
 U 1 1 5F99726C
 P 8575 3000
-F 0 "#PWR?" H 8575 2750 50  0001 C CNN
+F 0 "#PWR0103" H 8575 2750 50  0001 C CNN
 F 1 "GND" H 8580 2827 50  0000 C CNN
 F 2 "" H 8575 3000 50  0001 C CNN
@@
 Text Label 4500 2950 0    50   ~ 0
 pass
-Wire Wire Line
-	4725 2950 4525 2950
 Text Label 5775 3400 0    50   ~ 0
 pass
 $Comp
-L Device:R R?
+L Device:R R4
 U 1 1 5F99A37B
 P 6225 3250
-F 0 "R?" H 6295 3296 50  0000 L CNN
-F 1 "R" H 6295 3205 50  0000 L CNN
-F 2 "" V 6155 3250 50  0001 C CNN
+F 0 "R4" H 6295 3296 50  0000 L CNN
+F 1 "235k" H 6295 3205 50  0000 L CNN
+F 2 "Resistor_SMD:R_0603_1608Metric_Pad1.05x0.95mm_HandSolder" V 6155 3250 50  0001 C CNN
 F 3 "~" H 6225 3250 50  0001 C CNN
 	1    6225 3250
@@
 $EndComp
 $Comp
-L Device:R R?
+L Device:R R3
 U 1 1 5F99ABB4
 P 6225 2950
-F 0 "R?" H 6295 2996 50  0000 L CNN
-F 1 "R" H 6295 2905 50  0000 L CNN
-F 2 "" V 6155 2950 50  0001 C CNN
+F 0 "R3" H 6295 2996 50  0000 L CNN
+F 1 "100k" H 6295 2905 50  0000 L CNN
+F 2 "Resistor_SMD:R_0603_1608Metric_Pad1.05x0.95mm_HandSolder" V 6155 2950 50  0001 C CNN
 F 3 "~" H 6225 2950 50  0001 C CNN
 	1    6225 2950
@@
 	8575 2725 7825 2725
 $Comp
-L power:VCC #PWR?
+L power:VCC #PWR0104
 U 1 1 5F9896F1
 P 5225 2450
-F 0 "#PWR?" H 5225 2300 50  0001 C CNN
+F 0 "#PWR0104" H 5225 2300 50  0001 C CNN
 F 1 "VCC" H 5240 2623 50  0000 C CNN
 F 2 "" H 5225 2450 50  0001 C CNN
@@
 $EndComp
 $Comp
-L Isolator:LTV-817 U?
-U 1 1 5F9B065A
-P 2150 3075
-F 0 "U?" H 2150 3400 50  0000 C CNN
-F 1 "LTV-817" H 2150 3309 50  0000 C CNN
-F 2 "Package_DIP:DIP-4_W7.62mm" H 1950 2875 50  0001 L CIN
-F 3 "http://www.us.liteon.com/downloads/LTV-817-827-847.PDF" H 2150 2975 50  0001 L CNN
-	1    2150 3075
-	1    0    0    -1
-$EndComp
-$Comp
-L power:+12V #PWR?
+L power:+12V #PWR0105
 U 1 1 5F9B1391
 P 2625 2975
-F 0 "#PWR?" H 2625 2825 50  0001 C CNN
+F 0 "#PWR0105" H 2625 2825 50  0001 C CNN
 F 1 "+12V" H 2640 3148 50  0000 C CNN
 F 2 "" H 2625 2975 50  0001 C CNN
@@
 	2625 2975 2450 2975
 $Comp
-L power:GND #PWR?
+L power:GND #PWR0106
 U 1 1 5F9B2348
 P 2450 3750
-F 0 "#PWR?" H 2450 3500 50  0001 C CNN
+F 0 "#PWR0106" H 2450 3500 50  0001 C CNN
 F 1 "GND" H 2455 3577 50  0000 C CNN
 F 2 "" H 2450 3750 50  0001 C CNN
@@
 $EndComp
 $Comp
-L Device:R R?
+L Device:R R2
 U 1 1 5F9B2DED
 P 2450 3450
-F 0 "R?" H 2520 3496 50  0000 L CNN
+F 0 "R2" H 2520 3496 50  0000 L CNN
 F 1 "10k" H 2520 3405 50  0000 L CNN
-F 2 "" V 2380 3450 50  0001 C CNN
+F 2 "Resistor_SMD:R_0603_1608Metric_Pad1.05x0.95mm_HandSolder" V 2380 3450 50  0001 C CNN
 F 3 "~" H 2450 3450 50  0001 C CNN
 	1    2450 3450
@@
 	2450 3175 2450 3300
 $Comp
-L power:VCC #PWR?
+L power:VCC #PWR0107
 U 1 1 5F9B410B
 P 2850 3175
-F 0 "#PWR?" H 2850 3025 50  0001 C CNN
+F 0 "#PWR0107" H 2850 3025 50  0001 C CNN
 F 1 "VCC" H 2865 3348 50  0000 C CNN
 F 2 "" H 2850 3175 50  0001 C CNN
@@
 Text Label 2775 3175 2    50   ~ 0
 HV_ON
-Connection ~ 2450 3175
 Wire Wire Line
 	2450 3175 2850 3175
 $Comp
-L Device:C C?
+L Device:C C2
 U 1 1 5F9C368D
 P 5725 3725
-F 0 "C?" H 5840 3771 50  0000 L CNN
+F 0 "C2" H 5840 3771 50  0000 L CNN
 F 1 "1u" H 5840 3680 50  0000 L CNN
-F 2 "" H 5763 3575 50  0001 C CNN
+F 2 "Capacitor_SMD:C_0603_1608Metric_Pad1.05x0.95mm_HandSolder" H 5763 3575 50  0001 C CNN
 F 3 "~" H 5725 3725 50  0001 C CNN
 	1    5725 3725
@@
 Connection ~ 5725 3400
 $Comp
-L Device:C C?
+L Device:C C1
 U 1 1 5F9C8A14
 P 4650 3675
-F 0 "C?" H 4765 3721 50  0000 L CNN
+F 0 "C1" H 4765 3721 50  0000 L CNN
 F 1 "0.1u" H 4765 3630 50  0000 L CNN
-F 2 "" H 4688 3525 50  0001 C CNN
+F 2 "Capacitor_SMD:C_0603_1608Metric_Pad1.05x0.95mm_HandSolder" H 4688 3525 50  0001 C CNN
 F 3 "~" H 4650 3675 50  0001 C CNN
 	1    4650 3675
@@
 Wire Wire Line
 	4650 3875 5225 3875
+$Comp
+L Device:R R1
+U 1 1 5F9B78C3
+P 1850 2550
+F 0 "R1" H 1780 2504 50  0000 R CNN
+F 1 "39k" H 1780 2595 50  0000 R CNN
+F 2 "Resistor_THT:R_Axial_DIN0617_L17.0mm_D6.0mm_P30.48mm_Horizontal" V 1780 2550 50  0001 C CNN
+F 3 "~" H 1850 2550 50  0001 C CNN
+	1    1850 2550
+	1    0    0    1
+$EndComp
+Wire Wire Line
+	1850 2700 1850 2975
+$Comp
+L Connector_Generic:Conn_01x02 J1
+U 1 1 5F9BB97B
+P 1325 2325
+F 0 "J1" H 1243 2000 50  0000 C CNN
+F 1 "Conn_01x02" H 1243 2091 50  0000 C CNN
+F 2 "Connector_TE-Connectivity:TE_MATE-N-LOK_1-770866-x_1x02_P4.14mm_Vertical" H 1325 2325 50  0001 C CNN
+F 3 "~" H 1325 2325 50  0001 C CNN
+	1    1325 2325
+	-1   0    0    1
+$EndComp
+Wire Wire Line
+	1525 2225 1525 2275
+Wire Wire Line
+	1525 2275 1850 2275
+Wire Wire Line
+	1850 2275 1850 2400
+Connection ~ 1525 2275
+Wire Wire Line
+	1525 2275 1525 2325
+$Comp
+L Connector_Generic:Conn_01x02 J2
+U 1 1 5F9BEA2F
+P 1325 3225
+F 0 "J2" H 1243 2900 50  0000 C CNN
+F 1 "Conn_01x02" H 1243 2991 50  0000 C CNN
+F 2 "Connector_TE-Connectivity:TE_MATE-N-LOK_1-770866-x_1x02_P4.14mm_Vertical" H 1325 3225 50  0001 C CNN
+F 3 "~" H 1325 3225 50  0001 C CNN
+	1    1325 3225
+	-1   0    0    1
+$EndComp
+Wire Wire Line
+	1525 3125 1525 3175
+Wire Wire Line
+	1850 3175 1525 3175
+Connection ~ 1525 3175
+Wire Wire Line
+	1525 3175 1525 3225
+Text Label 1575 3175 0    50   ~ 0
+HV-
+Text Label 1625 2275 0    50   ~ 0
+HV+
+Wire Notes Line width 20
+	2200 4325 2200 1400
+Wire Notes Line width 20
+	2200 1400 975  1400
+Wire Notes Line width 20
+	975  1400 975  4325
+Wire Notes Line width 20
+	975  4325 2200 4325
+Text Notes 1350 1575 0    50   ~ 0
+High Voltage
+Wire Wire Line
+	4500 2950 4725 2950
+$Comp
+L Connector_Generic:Conn_01x02 J4
+U 1 1 5F9D59EC
+P 8775 3550
+F 0 "J4" H 8855 3542 50  0000 L CNN
+F 1 "Conn_01x02" H 8855 3451 50  0000 L CNN
+F 2 "Connector_TE-Connectivity:TE_MATE-N-LOK_1-770866-x_1x02_P4.14mm_Vertical" H 8775 3550 50  0001 C CNN
+F 3 "~" H 8775 3550 50  0001 C CNN
+	1    8775 3550
+	1    0    0    -1
+$EndComp
+$Comp
+L power:+12V #PWR0108
+U 1 1 5F9D6F6B
+P 8575 3550
+F 0 "#PWR0108" H 8575 3400 50  0001 C CNN
+F 1 "+12V" H 8590 3723 50  0000 C CNN
+F 2 "" H 8575 3550 50  0001 C CNN
+F 3 "" H 8575 3550 50  0001 C CNN
+	1    8575 3550
+	1    0    0    -1
+$EndComp
+$Comp
+L power:GND #PWR0109
+U 1 1 5F9D73CE
+P 8575 3650
+F 0 "#PWR0109" H 8575 3400 50  0001 C CNN
+F 1 "GND" H 8580 3477 50  0000 C CNN
+F 2 "" H 8575 3650 50  0001 C CNN
+F 3 "" H 8575 3650 50  0001 C CNN
+	1    8575 3650
+	1    0    0    -1
+$EndComp
+$Comp
+L Isolator:LTV-817S U1
+U 1 1 5F9DE7CE
+P 2150 3075
+F 0 "U1" H 2150 3400 50  0000 C CNN
+F 1 "LTV-817S" H 2150 3309 50  0000 C CNN
+F 2 "Package_DIP:SMDIP-4_W9.53mm" H 2150 2775 50  0001 C CNN
+F 3 "http://www.us.liteon.com/downloads/LTV-817-827-847.PDF" H 1800 3375 50  0001 C CNN
+	1    2150 3075
+	1    0    0    -1
+$EndComp
+Connection ~ 2450 3175
+$Comp
+L Mechanical:MountingHole H1
+U 1 1 5F9E7AA7
+P 1250 4950
+F 0 "H1" H 1350 4996 50  0000 L CNN
+F 1 "M3" H 1350 4905 50  0000 L CNN
+F 2 "MountingHole:MountingHole_3.2mm_M3" H 1250 4950 50  0001 C CNN
+F 3 "~" H 1250 4950 50  0001 C CNN
+	1    1250 4950
+	1    0    0    -1
+$EndComp
 $EndSCHEMATC
