File: Emrax_Breakout/Emrax_Breakout/Emrax_Breakout.sch (KiCad schematic (older format))
At the start: 3 parts

Commit message: Inital pcb layout
Parts:
- J1: renamed from J?; footprint (none) -> AERO_CUSTOM:TE_1-776276-1_8pin_Vertical
- J2: renamed from J?; footprint (none) -> Connector_JST:JST_PH_B2B-PH-K_1x02_P2.00mm_Vertical
- J3: renamed from J?; footprint (none) -> Connector_JST:JST_PH_B6B-PH-K_1x06_P2.00mm_Vertical
Changed lines of the file:
@@
 $EndDescr
 $Comp
-L Connector_Generic:Conn_01x08 J?
+L Connector_Generic:Conn_01x08 J1
 U 1 1 5FFBB53E
 P 3950 2975
-F 0 "J?" H 3868 2350 50  0000 C CNN
+F 0 "J1" H 3868 2350 50  0000 C CNN
 F 1 "Conn_01x08" H 3868 2441 50  0000 C CNN
-F 2 "" H 3950 2975 50  0001 C CNN
+F 2 "AERO_CUSTOM:TE_1-776276-1_8pin_Vertical" H 3950 2975 50  0001 C CNN
 F 3 "~" H 3950 2975 50  0001 C CNN
 	1    3950 2975
@@
 $EndComp
 $Comp
-L Connector_Generic:Conn_01x02 J?
+L Connector_Generic:Conn_01x02 J2
 U 1 1 5FFBC0C0
 P 5900 1950
-F 0 "J?" H 5980 1942 50  0000 L CNN
+F 0 "J2" H 5980 1942 50  0000 L CNN
 F 1 "Conn_01x02" H 5980 1851 50  0000 L CNN
-F 2 "" H 5900 1950 50  0001 C CNN
+F 2 "Connector_JST:JST_PH_B2B-PH-K_1x02_P2.00mm_Vertical" H 5900 1950 50  0001 C CNN
 F 3 "~" H 5900 1950 50  0001 C CNN
 	1    5900 1950
@@
 $EndComp
 $Comp
-L Connector_Generic:Conn_01x06 J?
+L Connector_Generic:Conn_01x06 J3
 U 1 1 5FFBC89E
 P 5975 3150
-F 0 "J?" H 5893 2625 50  0000 C CNN
+F 0 "J3" H 5893 2625 50  0000 C CNN
 F 1 "Conn_01x06" H 5893 2716 50  0000 C CNN
-F 2 "" H 5975 3150 50  0001 C CNN
+F 2 "Connector_JST:JST_PH_B6B-PH-K_1x06_P2.00mm_Vertical" H 5975 3150 50  0001 C CNN
 F 3 "~" H 5975 3150 50  0001 C CNN
 	1    5975 3150
@@
 	4450 3175 4150 3175
 $Comp
-L power:GND #PWR?
+L power:GND #PWR0101
 U 1 1 5FFC988D
 P 4450 3275
-F 0 "#PWR?" H 4450 3025 50  0001 C CNN
+F 0 "#PWR0101" H 4450 3025 50  0001 C CNN
 F 1 "GND" H 4455 3102 50  0000 C CNN
 F 2 "" H 4450 3275 50  0001 C CNN
@@
 SIN-
 $Comp
-L power:GND #PWR?
+L power:GND #PWR0102
 U 1 1 5FFCB11A
 P 5500 3350
-F 0 "#PWR?" H 5500 3100 50  0001 C CNN
+F 0 "#PWR0102" H 5500 3100 50  0001 C CNN
 F 1 "GND" H 5505 3177 50  0000 C CNN
 F 2 "" H 5500 3350 50  0001 C CNN
