File: DaqBoard/KiCad/DaqBoard.sch (KiCad schematic (older format))
At the start: 20 parts

Commit message: initial pcb layout
Parts:
- removed Q? (x2): PSMN5R2-60YL, Package_TO_SOT_SMD:LFPAK56, symbol Transistor_FET:PSMN5R2-60YL
- added Q? (x2): PSMN5R2-60YL, Package_TO_SOT_SMD:LFPAK56, symbol Transistor_FET:PSMN5R2-60YL
Connections:
- net BRAKE_OUT: now also Q?.5 (D)
- net BRAKE_SIG: now also Q?.4 (G)
- net FAN_OUT: now also Q?.5 (D)
- net FAN_SIG: now also Q?.4 (G)
- net GND: now also Q?.1 (S), Q?.1 (S), Q?.2 (S), Q?.2 (S), Q?.3 (S), Q?.3 (S)
Changed lines of the file:
@@
 	6800 7150 6550 7150
 $Comp
-L power:GND #PWR?
+L power:GND #PWR0101
 U 1 1 5FFCBDFC
 P 6800 7150
-F 0 "#PWR?" H 6800 6900 50  0001 C CNN
+F 0 "#PWR0101" H 6800 6900 50  0001 C CNN
 F 1 "GND" H 6805 6977 50  0000 C CNN
 F 2 "" H 6800 7150 50  0001 C CNN
@@
 	6800 6950 6550 6950
 $Comp
-L power:+5V #PWR?
+L power:+5V #PWR0102
 U 1 1 5FFC8CD6
 P 6800 6950
-F 0 "#PWR?" H 6800 6800 50  0001 C CNN
+F 0 "#PWR0102" H 6800 6800 50  0001 C CNN
 F 1 "+5V" H 6815 7123 50  0000 C CNN
 F 2 "" H 6800 6950 50  0001 C CNN
@@
 	4550 7400 4050 7400
 $Comp
-L power:GND #PWR?
+L power:GND #PWR0103
 U 1 1 5FFC8CD4
 P 4550 7400
-F 0 "#PWR?" H 4550 7150 50  0001 C CNN
+F 0 "#PWR0103" H 4550 7150 50  0001 C CNN
 F 1 "GND" H 4555 7227 50  0000 C CNN
 F 2 "" H 4550 7400 50  0001 C CNN
@@
 Connection ~ 5000 6825
 $Comp
-L power:+5V #PWR?
+L power:+5V #PWR0104
 U 1 1 5FFC068A
 P 5000 6825
-F 0 "#PWR?" H 5000 6675 50  0001 C CNN
+F 0 "#PWR0104" H 5000 6675 50  0001 C CNN
 F 1 "+5V" H 5015 6998 50  0000 C CNN
 F 2 "" H 5000 6825 50  0001 C CNN
@@
 Connection ~ 4050 6825
 $Comp
-L power:+12V #PWR?
+L power:+12V #PWR0105
 U 1 1 5FFBFE26
 P 3500 6825
-F 0 "#PWR?" H 3500 6675 50  0001 C CNN
+F 0 "#PWR0105" H 3500 6675 50  0001 C CNN
 F 1 "+12V" H 3450 7000 50  0000 C CNN
 F 2 "" H 3500 6825 50  0001 C CNN
@@
 Connection ~ 2225 2275
 $Comp
-L power:+5V #PWR?
+L power:+5V #PWR0106
 U 1 1 5FFB5286
 P 2225 2150
-F 0 "#PWR?" H 2225 2000 50  0001 C CNN
+F 0 "#PWR0106" H 2225 2000 50  0001 C CNN
 F 1 "+5V" H 2240 2323 50  0000 C CNN
 F 2 "" H 2225 2150 50  0001 C CNN
@@
 	1025 2575 1025 2725
 $Comp
-L power:GND #PWR?
+L power:GND #PWR0107
 U 1 1 5FFB6133
 P 1025 3025
-F 0 "#PWR?" H 1025 2775 50  0001 C CNN
+F 0 "#PWR0107" H 1025 2775 50  0001 C CNN
 F 1 "GND" H 1030 2852 50  0000 C CNN
 F 2 "" H 1025 3025 50  0001 C CNN
@@
 $EndComp
 $Comp
-L power:GND #PWR?
+L power:GND #PWR0108
 U 1 1 5FFB6516
 P 825 2450
-F 0 "#PWR?" H 825 2200 50  0001 C CNN
+F 0 "#PWR0108" H 825 2200 50  0001 C CNN
 F 1 "GND" H 830 2277 50  0000 C CNN
 F 2 "" H 825 2450 50  0001 C CNN
@@
 Connection ~ 2225 2150
 $Comp
-L power:GND #PWR?
+L power:GND #PWR0109
 U 1 1 5FFBB4A3
 P 2175 5275
-F 0 "#PWR?" H 2175 5025 50  0001 C CNN
+F 0 "#PWR0109" H 2175 5025 50  0001 C CNN
 F 1 "GND" H 2180 5102 50  0000 C CNN
 F 2 "" H 2175 5275 50  0001 C CNN
@@
 $EndComp
 $Comp
-L power:GND #PWR?
+L power:GND #PWR0110
 U 1 1 5FFBBD1B
 P 5600 6825
-F 0 "#PWR?" H 5600 6575 50  0001 C CNN
+F 0 "#PWR0110" H 5600 6575 50  0001 C CNN
 F 1 "GND" H 5605 6652 50  0000 C CNN
 F 2 "" H 5600 6825 50  0001 C CNN
@@
 Wire Wire Line
 	3300 4675 2775 4675
-$Comp
-L Transistor_FET:PSMN5R2-60YL Q?
-U 1 1 6001EA29
-P 5325 5250
-F 0 "Q?" H 5530 5296 50  0000 L CNN
-F 1 "PSMN5R2-60YL" H 5530 5205 50  0000 L CNN
-F 2 "Package_TO_SOT_SMD:LFPAK56" H 5475 5250 50  0001 C CNN
-F 3 "https://assets.nexperia.com/documents/data-sheet/PSMN5R2-60YL.pdf" H 5325 5250 50  0001 C CNN
-	1    5325 5250
-	1    0    0    -1
-$EndComp
 Text Label 4500 5250 0    50   ~ 0
 BRAKE_SIG
@@
 	5675 5050 5425 5050
 $Comp
-L power:GND #PWR?
+L power:GND #PWR0111
 U 1 1 600242C5
 P 5425 5725
-F 0 "#PWR?" H 5425 5475 50  0001 C CNN
+F 0 "#PWR0111" H 5425 5475 50  0001 C CNN
 F 1 "GND" H 5430 5552 50  0000 C CNN
 F 2 "" H 5425 5725 50  0001 C CNN
@@
 Wire Wire Line
 	5425 5625 5425 5725
-$Comp
-L Transistor_FET:PSMN5R2-60YL Q?
-U 1 1 6002C7AF
-P 7375 5275
-F 0 "Q?" H 7580 5321 50  0000 L CNN
-F 1 "PSMN5R2-60YL" H 7580 5230 50  0000 L CNN
-F 2 "Package_TO_SOT_SMD:LFPAK56" H 7525 5275 50  0001 C CNN
-F 3 "https://assets.nexperia.com/documents/data-sheet/PSMN5R2-60YL.pdf" H 7375 5275 50  0001 C CNN
-	1    7375 5275
-	1    0    0    -1
-$EndComp
 Text Label 6550 5275 0    50   ~ 0
 FAN_SIG
@@
 	7725 5075 7475 5075
 $Comp
-L power:GND #PWR?
+L power:GND #PWR0112
 U 1 1 6002C7BD
 P 7475 5750
-F 0 "#PWR?" H 7475 5500 50  0001 C CNN
+F 0 "#PWR0112" H 7475 5500 50  0001 C CNN
 F 1 "GND" H 7480 5577 50  0000 C CNN
 F 2 "" H 7475 5750 50  0001 C CNN
@@
 	9825 3800 9825 3700
 $Comp
-L power:+12V #PWR?
+L power:+12V #PWR0113
 U 1 1 600AA4CA
 P 9850 2600
-F 0 "#PWR?" H 9850 2450 50  0001 C CNN
+F 0 "#PWR0113" H 9850 2450 50  0001 C CNN
 F 1 "+12V" H 9865 2773 50  0000 C CNN
 F 2 "" H 9850 2600 50  0001 C CNN
@@
 	9850 2600 10250 2600
 $Comp
-L power:GND #PWR?
+L power:GND #PWR0114
 U 1 1 600B1C71
 P 9850 4800
-F 0 "#PWR?" H 9850 4550 50  0001 C CNN
+F 0 "#PWR0114" H 9850 4550 50  0001 C CNN
 F 1 "GND" H 9855 4627 50  0000 C CNN
 F 2 "" H 9850 4800 50  0001 C CNN
@@
 	9825 4000 10250 4000
 $Comp
-L power:+5V #PWR?
+L power:+5V #PWR0115
 U 1 1 600C423E
 P 9675 4100
-F 0 "#PWR?" H 9675 3950 50  0001 C CNN
+F 0 "#PWR0115" H 9675 3950 50  0001 C CNN
 F 1 "+5V" H 9690 4273 50  0000 C CNN
 F 2 "" H 9675 4100 50  0001 C CNN
@@
 	1    0    0    -1
 $EndComp
+$Comp
+L Transistor_FET:PSMN5R2-60YL Q?
+U 1 1 5FFDB6AD
+P 5325 5250
+F 0 "Q?" H 5530 5296 50  0000 L CNN
+F 1 "PSMN5R2-60YL" H 5530 5205 50  0000 L CNN
+F 2 "Package_TO_SOT_SMD:LFPAK56" H 5475 5250 50  0001 C CNN
+F 3 "https://assets.nexperia.com/documents/data-sheet/PSMN5R2-60YL.pdf" H 5325 5250 50  0001 C CNN
+	1    5325 5250
+	1    0    0    -1
+$EndComp
+$Comp
+L Transistor_FET:PSMN5R2-60YL Q?
+U 1 1 5FFDE8F8
+P 7375 5275
+F 0 "Q?" H 7580 5321 50  0000 L CNN
+F 1 "PSMN5R2-60YL" H 7580 5230 50  0000 L CNN
+F 2 "Package_TO_SOT_SMD:LFPAK56" H 7525 5275 50  0001 C CNN
+F 3 "https://assets.nexperia.com/documents/data-sheet/PSMN5R2-60YL.pdf" H 7375 5275 50  0001 C CNN
+	1    7375 5275
+	1    0    0    -1
+$EndComp

Commit message: inital layouts
Parts:
- C1, C2, C3, C4: renamed from C?; footprint (none) -> Capacitor_SMD:C_0603_1608Metric_Pad1.08x0.95mm_HandSolder
- D1: renamed from D?; footprint (none) -> LED_SMD:LED_0603_1608Metric_Pad1.05x0.95mm_HandSolder
- F1: renamed from F?; footprint (none) -> Fuse:Fuse_1812_4532Metric_Pad1.30x3.40mm_HandSolder
- H1, H2: renamed from H?; footprint (none) -> MountingHole:MountingHole_3.2mm_M3
- J1, J4: renamed from J?; footprint (none) -> AERO_CUSTOM:RJ45_TE_5569284-1-8P8CX_Vertical
- J2: renamed from J?; footprint (none) -> Connector_PinHeader_2.54mm:PinHeader_1x02_P2.54mm_Vertical
- J3: renamed from J?; footprint (none) -> Connector_PinHeader_2.54mm:PinHeader_2x03_P2.54mm_Vertical
- J5: renamed from J?; footprint (none) -> AERO_CUSTOM:TE_1-770669-1_23pin_Horizontal
- R1, R2, R3: renamed from R?; footprint (none) -> Resistor_SMD:R_0603_1608Metric_Pad0.98x0.95mm_HandSolder
- gave numbers to parts that had none: 4
Connections:
- net +12V: now also J5.16 (Pin_16); no longer J5.1 (Pin_1)
- net +5V: now also J5.1 (Pin_1), J5.2 (Pin_2), J5.3 (Pin_3), J5.4 (Pin_4), J5.5 (Pin_5); no longer J5.16 (Pin_16), J5.17 (Pin_17), J5.18 (Pin_18), J5.19 (Pin_19), J5.20 (Pin_20)
- net BRAKE_OUT: now also J5.23 (Pin_23); no longer J5.14 (Pin_14)
- net CANH: now also J5.18 (Pin_18); no longer J5.11 (Pin_11)
- net CANL: now also J5.17 (Pin_17), J5.9 (Pin_9); no longer J5.12 (Pin_12), J5.13 (Pin_13)
- net DAMPER_L: now also J5.11 (Pin_11); no longer J5.4 (Pin_4)
- net DAMPER_R: now also J5.12 (Pin_12); no longer J5.5 (Pin_5)
- net GND: now also J5.6 (Pin_6), J5.7 (Pin_7), J5.8 (Pin_8); no longer J5.21 (Pin_21), J5.22 (Pin_22), J5.23 (Pin_23)
- net SENSOR_1: now also J5.13 (Pin_13); no longer J5.6 (Pin_6)
- net SENSOR_2: now also J5.14 (Pin_14); no longer J5.7 (Pin_7)
- net SENSOR_3: now also J5.21 (Pin_21); no longer J5.8 (Pin_8)
- net SENSOR_4: now also J5.22 (Pin_22); no longer J5.9 (Pin_9)
- net WHEEL_L: now also J5.19 (Pin_19); no longer J5.2 (Pin_2)
- net WHEEL_R: now also J5.20 (Pin_20); no longer J5.3 (Pin_3)
Other:
- moved on the sheet: J5

Commit message: first layout design
Parts:
- removed H1, H2: MountingHole, MountingHole:MountingHole_3.2mm_M3, symbol Mechanical:MountingHole
Connections:
- net +5V: now also J5.10 (Pin_10), J5.11 (Pin_11), J5.17 (Pin_17), J5.18 (Pin_18), J5.9 (Pin_9); no longer J5.1 (Pin_1), J5.2 (Pin_2), J5.3 (Pin_3), J5.4 (Pin_4), J5.5 (Pin_5)
- net BRAKE_OUT: now also J5.22 (Pin_22); no longer J5.23 (Pin_23)
- net BRAKE_SIG: now also U1.2 (PD4); no longer U1.1 (PD3)
- net DAMPER_L: now also J5.14 (Pin_14); no longer J5.11 (Pin_11)
- net DAMPER_R: now also J5.15 (Pin_15); no longer J5.12 (Pin_12)
- net FAN_OUT: now also J5.21 (Pin_21); no longer J5.15 (Pin_15)
- net FAN_SIG: now also U1.1 (PD3); no longer U1.2 (PD4)
- net GND: now also J5.1 (Pin_1), J5.2 (Pin_2), J5.3 (Pin_3); no longer J5.6 (Pin_6), J5.7 (Pin_7), J5.8 (Pin_8)
- net SENSOR_1: now also J5.7 (Pin_7); no longer J5.13 (Pin_13)
- net SENSOR_2: now also J5.8 (Pin_8); no longer J5.14 (Pin_14)
- net SENSOR_3: now also J5.6 (Pin_6); no longer J5.21 (Pin_21)
- net SENSOR_4: now also J5.5 (Pin_5); no longer J5.22 (Pin_22)
- net WHEEL_L: now also J5.4 (Pin_4); no longer J5.19 (Pin_19)
- net WHEEL_R: now also J5.23 (Pin_23); no longer J5.20 (Pin_20)
- removed net CANH: J2.2 (Pin_2), J5.10 (Pin_10), J5.18 (Pin_18)
- removed net CANL: J2.1 (Pin_1), J5.17 (Pin_17), J5.9 (Pin_9)
- new net CAN+: J2.2 (Pin_2), J5.12 (Pin_12), J5.19 (Pin_19)
- new net CAN-: J2.1 (Pin_1), J5.13 (Pin_13), J5.20 (Pin_20)
Changed lines of the file:
@@
 	1825 7225 2150 7225
 Text Label 3375 7050 2    50   ~ 0
-CANH
+CAN+
 Text Label 3375 7200 2    50   ~ 0
-CANL
+CAN-
 Wire Wire Line
 	3375 7050 3150 7050
@@
 Wire Wire Line
 	3200 3775 2775 3775
+Text Label 3300 4675 2    50   ~ 0
+BRAKE_SIG
+Wire Wire Line
+	3300 4575 2775 4575
 Text Label 3300 4575 2    50   ~ 0
-BRAKE_SIG
-Wire Wire Line
-	3300 4575 2775 4575
-Text Label 3300 4675 2    50   ~ 0
 FAN_SIG
 Wire Wire Line
@@
 Wire Wire Line
 	3200 3975 2775 3975
-Text Label 10050 4225 0    50   ~ 0
+Text Label 10050 2725 0    50   ~ 0
 WHEEL_L
-Text Label 10050 4325 0    50   ~ 0
+Text Label 10050 4625 0    50   ~ 0
 WHEEL_R
 Wire Wire Line
-	10475 4325 10050 4325
-Wire Wire Line
-	10050 4225 10475 4225
-Text Label 10050 3425 0    50   ~ 0
+	10475 4625 10050 4625
+Wire Wire Line
+	10050 2725 10475 2725
+Text Label 10050 3725 0    50   ~ 0
 DAMPER_L
 Wire Wire Line
-	10050 3425 10475 3425
-Text Label 10050 3525 0    50   ~ 0
+	10050 3725 10475 3725
+Text Label 10050 3825 0    50   ~ 0
 DAMPER_R
 Wire Wire Line
-	10050 3525 10475 3525
-Text Label 10050 4425 0    50   ~ 0
+	10050 3825 10475 3825
+Text Label 10050 2925 0    50   ~ 0
 SENSOR_3
 Wire Wire Line
-	10050 4425 10475 4425
-Text Label 10050 4525 0    50   ~ 0
+	10475 2925 10050 2925
+Text Label 10050 2825 0    50   ~ 0
 SENSOR_4
 Wire Wire Line
-	10050 4525 10475 4525
-Text Label 10050 3625 0    50   ~ 0
+	10475 2825 10050 2825
+Text Label 10050 3025 0    50   ~ 0
 SENSOR_1
 Wire Wire Line
-	10050 3625 10475 3625
-Text Label 10050 3725 0    50   ~ 0
+	10475 3125 10050 3125
+Text Label 10050 3125 0    50   ~ 0
 SENSOR_2
 Wire Wire Line
-	10050 3725 10475 3725
-Text Label 10000 3325 0    50   ~ 0
-CANH
-Text Label 10000 3225 0    50   ~ 0
-CANL
+	10475 3025 10050 3025
+Text Label 10000 4225 0    50   ~ 0
+CAN+
+Text Label 10000 4325 0    50   ~ 0
+CAN-
 $Comp
 L power:+12V #PWR0113
 U 1 1 600AA4CA
-P 9775 3925
-F 0 "#PWR0113" H 9775 3775 50  0001 C CNN
-F 1 "+12V" H 9790 4098 50  0000 C CNN
-F 2 "" H 9775 3925 50  0001 C CNN
-F 3 "" H 9775 3925 50  0001 C CNN
-	1    9775 3925
-	1    0    0    -1
-$EndComp
-Wire Wire Line
-	9775 3925 10475 3925
+P 9925 3925
+F 0 "#PWR0113" H 9925 3775 50  0001 C CNN
+F 1 "+12V" H 9940 4098 50  0000 C CNN
+F 2 "" H 9925 3925 50  0001 C CNN
+F 3 "" H 9925 3925 50  0001 C CNN
+	1    9925 3925
+	1    0    0    -1
+$EndComp
+Wire Wire Line
+	9925 3925 10475 3925
 $Comp
 L power:GND #PWR0114
 U 1 1 600B1C71
-P 9775 3125
-F 0 "#PWR0114" H 9775 2875 50  0001 C CNN
-F 1 "GND" H 9780 2952 50  0000 C CNN
-F 2 "" H 9775 3125 50  0001 C CNN
-F 3 "" H 9775 3125 50  0001 C CNN
-	1    9775 3125
-	1    0    0    -1
-$EndComp
-Text Label 10025 4625 0    50   ~ 0
+P 9775 2625
+F 0 "#PWR0114" H 9775 2375 50  0001 C CNN
+F 1 "GND" H 9780 2452 50  0000 C CNN
+F 2 "" H 9775 2625 50  0001 C CNN
+F 3 "" H 9775 2625 50  0001 C CNN
+	1    9775 2625
+	1    0    0    -1
+$EndComp
+Text Label 10025 4525 0    50   ~ 0
 BRAKE_OUT
-Text Label 10025 3825 0    50   ~ 0
+Text Label 10025 4425 0    50   ~ 0
 FAN_OUT
 $Comp
 L power:+5V #PWR0115
 U 1 1 600C423E
-P 9775 2425
-F 0 "#PWR0115" H 9775 2275 50  0001 C CNN
-F 1 "+5V" H 9790 2598 50  0000 C CNN
-F 2 "" H 9775 2425 50  0001 C CNN
-F 3 "" H 9775 2425 50  0001 C CNN
-	1    9775 2425
-	1    0    0    -1
-$EndComp
-Wire Wire Line
-	9775 2525 9775 2425
-Connection ~ 9775 2425
-Wire Wire Line
-	9775 2625 9775 2525
+P 9775 3225
+F 0 "#PWR0115" H 9775 3075 50  0001 C CNN
+F 1 "+5V" H 9790 3398 50  0000 C CNN
+F 2 "" H 9775 3225 50  0001 C CNN
+F 3 "" H 9775 3225 50  0001 C CNN
+	1    9775 3225
+	1    0    0    -1
+$EndComp
+Wire Wire Line
+	9775 2525 9775 2625
+Connection ~ 9775 2625
+Wire Wire Line
+	9775 2425 9775 2525
 Connection ~ 9775 2525
-Wire Wire Line
-	9775 2725 9775 2625
-Connection ~ 9775 2625
-Wire Wire Line
-	9775 3025 9775 3125
-Connection ~ 9775 3125
-Wire Wire Line
-	9775 2925 9775 3025
-Connection ~ 9775 3025
-Wire Wire Line
-	9775 2825 9775 2725
-Connection ~ 9775 2725
 $Comp
 L Connector:RJ45 J4
@@
 $EndComp
 Text Label 5775 2475 0    50   ~ 0
-CANH
+CAN+
 Text Label 5775 2375 0    50   ~ 0
-CANL
+CAN-
 Wire Wire Line
 	5775 2475 6000 2475
@@
 	5700 2575 5700 2050
 $Comp
-L Mechanical:MountingHole H2
-U 1 1 60178799
-P 750 6975
-F 0 "H2" H 850 7021 50  0000 L CNN
-F 1 "MountingHole" H 850 6930 50  0000 L CNN
-F 2 "MountingHole:MountingHole_3.2mm_M3" H 750 6975 50  0001 C CNN
-F 3 "~" H 750 6975 50  0001 C CNN
-	1    750  6975
-	1    0    0    -1
-$EndComp
-$Comp
-L Mechanical:MountingHole H1
-U 1 1 60178F9F
-P 725 7500
-F 0 "H1" H 825 7546 50  0000 L CNN
-F 1 "MountingHole" H 825 7455 50  0000 L CNN
-F 2 "MountingHole:MountingHole_3.2mm_M3" H 725 7500 50  0001 C CNN
-F 3 "~" H 725 7500 50  0001 C CNN
-	1    725  7500
-	1    0    0    -1
-$EndComp
-$Comp
 L Transistor_FET:PSMN5R2-60YL Q1
 U 1 1 5FFDB6AD
@@
 $EndComp
 Wire Wire Line
-	9775 2925 10475 2925
-Wire Wire Line
-	9775 3025 10475 3025
-Wire Wire Line
-	9775 3125 10475 3125
-Wire Wire Line
-	9775 2825 10475 2825
-Wire Wire Line
-	9775 2725 10475 2725
+	9775 2425 10475 2425
+Wire Wire Line
+	9775 2525 10475 2525
 Wire Wire Line
 	9775 2625 10475 2625
 Wire Wire Line
-	9775 2525 10475 2525
-Wire Wire Line
-	9775 2425 10475 2425
-Text Label 10025 4025 0    50   ~ 0
-CANL
-Text Label 10025 4125 0    50   ~ 0
-CANH
-Wire Wire Line
-	10000 3225 10475 3225
-Wire Wire Line
-	10000 3325 10475 3325
-Wire Wire Line
-	10025 3825 10475 3825
-Wire Wire Line
-	10025 4025 10475 4025
-Wire Wire Line
-	10025 4125 10475 4125
-Wire Wire Line
-	10025 4625 10475 4625
+	9775 4125 10475 4125
+Wire Wire Line
+	9775 4025 10475 4025
+Wire Wire Line
+	9775 3425 10475 3425
+Wire Wire Line
+	9775 3325 10475 3325
+Wire Wire Line
+	9775 3225 10475 3225
+Text Label 10025 3625 0    50   ~ 0
+CAN-
+Text Label 10025 3525 0    50   ~ 0
+CAN+
+Wire Wire Line
+	10000 4225 10475 4225
+Wire Wire Line
+	10000 4325 10475 4325
+Wire Wire Line
+	10025 4425 10475 4425
+Wire Wire Line
+	10025 4525 10475 4525
+Wire Wire Line
+	9775 3225 9775 3325
+Connection ~ 9775 3225
+Connection ~ 9775 3325
+Wire Wire Line
+	9775 3325 9775 3425
+$Comp
+L power:+5V #PWR0124
+U 1 1 6006A34A
+P 9775 4025
+F 0 "#PWR0124" H 9775 3875 50  0001 C CNN
+F 1 "+5V" H 9790 4198 50  0000 C CNN
+F 2 "" H 9775 4025 50  0001 C CNN
+F 3 "" H 9775 4025 50  0001 C CNN
+	1    9775 4025
+	1    0    0    -1
+$EndComp
+Wire Wire Line
+	9775 4025 9775 4125
+Connection ~ 9775 4025
+Text Label 1825 7425 0    50   ~ 0
+CAN_INT
+Wire Wire Line
+	1825 7425 2150 7425
+Wire Wire Line
+	10025 3625 10475 3625
+Wire Wire Line
+	10025 3525 10475 3525
 $EndSCHEMATC

Commit message: update PCB Layout
Connections:
- net SENSOR_3: no longer J5.6 (Pin_6)
- net SENSOR_4: no longer J5.5 (Pin_5)
- net SENSOR_5: now also J5.5 (Pin_5)
- net SENSOR_6: now also J5.6 (Pin_6)
Other:
- note added: "analog\n"
- note added: "digital"
Changed lines of the file:
@@
 	10050 3825 10475 3825
 Text Label 10050 2925 0    50   ~ 0
-SENSOR_3
+SENSOR_6
 Wire Wire Line
 	10475 2925 10050 2925
 Text Label 10050 2825 0    50   ~ 0
-SENSOR_4
+SENSOR_5
 Wire Wire Line
 	10475 2825 10050 2825
@@
 Wire Wire Line
 	10025 3525 10475 3525
+Text Notes 10800 2800 0    50   ~ 0
+analog\n
+Text Notes 10800 2900 0    50   ~ 0
+analog\n
+Text Notes 10800 3000 0    50   ~ 0
+digital
+Text Notes 10800 3100 0    50   ~ 0
+digital
 $EndSCHEMATC

Commit message: notes from design review 1
Connections:
- net BRAKE_SIG: now also U1.13 (PB1); no longer U1.2 (PD4)
- net SENSOR_4: now also U1.14 (PB2); no longer U1.13 (PB1)
Other:
- note added: "PWM"
Changed lines of the file:
@@
 Wire Wire Line
 	3200 3775 2775 3775
-Text Label 3300 4675 2    50   ~ 0
+Text Label 3300 2675 2    50   ~ 0
 BRAKE_SIG
 Wire Wire Line
@@
 FAN_SIG
 Wire Wire Line
-	3300 4675 2775 4675
+	3300 2675 2775 2675
 Text Label 4500 5250 0    50   ~ 0
 BRAKE_SIG
@@
 Wire Wire Line
 	3200 2575 2775 2575
-Text Label 3200 2675 2    50   ~ 0
+Text Label 3200 2775 2    50   ~ 0
 SENSOR_4
 Wire Wire Line
-	3200 2675 2775 2675
+	3200 2775 2775 2775
 Text Label 3200 3875 2    50   ~ 0
 SENSOR_5
@@
 Text Notes 10800 3100 0    50   ~ 0
 digital
+Text Notes 3525 4575 2    50   ~ 0
+PWM
+Text Notes 3500 2675 2    50   ~ 0
+PWM
 $EndSCHEMATC
