File: DaqBoard/KiCad/DaqBoard.kicad_pcb (KiCad board)
At the start: 2 copper layers, 27 parts, among them J1 RJ45, J2 Conn_01x02, J3 Conn_02x03_Odd_Even, J4 RJ45, J5 Conn_01x23, Q1 PSMN5R2-60YL, Q2 PSMN5R2-60YL, U1 ATmega328P-AU, U2 R-785.0-1.0, U3 MCP2515-xSO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

Commit message: first layout design
Parts:
- removed H1, H2: MountingHole, MountingHole:MountingHole_3.2mm_M3
- added G***: LOGO, AERO_CUSTOM:AERO_Logo_10x4mm, F.Cu at (154.0, 108.6)
- C2, C3, C4, C6, F1, R1, R3, R5, U3, U4: moved to B.Cu
- moved J4 49.1 mm to (146.7, 102.3), turned to 90 degrees
- moved R3 30.9 mm to (141.2, 98.4), turned to 270 degrees
- moved C4 28.1 mm to (136.4, 102.4), turned to 270 degrees
- moved C3 23.7 mm to (136.4, 105.9), turned to 90 degrees
- moved C6 22.5 mm to (128.7, 91.8), turned to 90 degrees
- moved R1 21.7 mm to (135.1, 98.6), turned to 270 degrees
- moved Q1 21.0 mm to (132.7, 92.5)
- moved Q2 19.9 mm to (139.2, 92.5), turned to 90 degrees
- moved R2 19.8 mm to (144.3, 107.2), turned to 180 degrees
- moved D1 17.9 mm to (144.3, 109.7)
- moved Y1 15.7 mm to (128.4, 108.1), turned to 270 degrees
- moved U2 15.1 mm to (139.7, 107.3)
- moved J2 13.5 mm to (143.4, 85.9), turned to 90 degrees
- moved U3 13.0 mm to (128.3, 104.8), turned to 180 degrees
- moved R5 12.9 mm to (136.9, 85.9), turned to 135 degrees
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Connections:
- J2 pad 1: /CANL -> /CAN-
- J2 pad 2: /CANH -> /CAN+
- J5 pad 1: +5V -> GND
- J5 pad 10: /CANH -> +5V
- J5 pad 11: /DAMPER_L -> +5V
- J5 pad 12: /DAMPER_R -> /CAN+
- J5 pad 13: /SENSOR_1 -> /CAN-
- J5 pad 14: /SENSOR_2 -> /DAMPER_L
- J5 pad 15: /FAN_OUT -> /DAMPER_R
- J5 pad 17: /CANL -> +5V
- J5 pad 18: /CANH -> +5V
- J5 pad 19: /WHEEL_L -> /CAN+
- J5 pad 2: +5V -> GND
- J5 pad 20: /WHEEL_R -> /CAN-
- J5 pad 21: /SENSOR_3 -> /FAN_OUT
- J5 pad 22: /SENSOR_4 -> /BRAKE_OUT
- J5 pad 23: /BRAKE_OUT -> /WHEEL_R
- J5 pad 3: +5V -> GND
- J5 pad 4: +5V -> /WHEEL_L
- J5 pad 5: +5V -> /SENSOR_4
- J5 pad 6: GND -> /SENSOR_3
- J5 pad 7: GND -> /SENSOR_1
- J5 pad 8: GND -> /SENSOR_2
- J5 pad 9: /CANL -> +5V
- R5 pad 1: /CANH -> /CAN+
- R5 pad 2: /CANL -> /CAN-
- U1 pad 1: /BRAKE_SIG -> /FAN_SIG
- U1 pad 2: /FAN_SIG -> /BRAKE_SIG
- U4 pad 6: /CANL -> /CAN-
- U4 pad 7: /CANH -> /CAN+
Routing:
- net +5V: track 0.00 -> 130.7 mm, vias 0 -> 2
- net /WHEEL_L: track 0.00 -> 45.1 mm, vias 0 -> 1
- net /SENSOR_4: track 0.00 -> 43.3 mm, vias 0 -> 1
- net Net-(C3-Pad1): track 0.00 -> 42.0 mm
- net /SENSOR_3: track 0.00 -> 39.1 mm, vias 0 -> 1
- net /SENSOR_1: track 0.00 -> 33.3 mm, vias 0 -> 1
- net /FAN_SIG: track 0.00 -> 29.3 mm, vias 0 -> 1
- net /DAMPER_L: track 0.00 -> 29.2 mm, vias 0 -> 1
- net /E4_P: track 0.00 -> 28.7 mm
- net /E4_N: track 0.00 -> 28.7 mm
- net /SENSOR_2: track 0.00 -> 27.7 mm, vias 0 -> 1
- net /CAN-: track 0.00 -> 27.7 mm
- net /E1_P: track 0.00 -> 27.4 mm
- net /E1_N: track 0.00 -> 27.4 mm
- net /E3_P: track 0.00 -> 27.3 mm
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- added copper zone on B.Cu, net +5V
- added copper zone on F.Cu, net /BRAKE_OUT
- added copper zone on F.Cu, net /FAN_OUT
- added copper zone on B.Cu, net GND
- added copper zone on F.Cu, net GND
Other:
- board outline added: 61 x 41.3 mm
- board text added: "DAQ G.SPEARING 21.012"

Commit message: update PCB Layout
Parts:
- removed G***: LOGO, AERO_CUSTOM:AERO_Logo_10x4mm
- moved C1 5.82 mm to (116.8, 87.4), turned to 180 degrees
- moved U1 0.95 mm to (118.0, 94.9)
Connections:
- J5 pad 5: /SENSOR_4 -> /SENSOR_5
- J5 pad 6: /SENSOR_3 -> /SENSOR_6
- U1 pad 12: /SENSOR_3 -> (no net)
- U1 pad 13: /SENSOR_4 -> (no net)
- U1 pad 27: (no net) -> /SENSOR_5
- U1 pad 28: (no net) -> /SENSOR_6
Routing:
- net /SENSOR_4: track 43.3 -> 0.00 mm, vias 1 -> 0
- net /SENSOR_3: track 39.1 -> 0.00 mm, vias 1 -> 0
- net /SENSOR_5: track 0.00 -> 36.4 mm, vias 0 -> 1
- net /SENSOR_6: track 0.00 -> 31.8 mm, vias 0 -> 1
- net /RESET: track 19.2 -> 34.8 mm
- net GND: track 11.9 -> 4.53 mm, vias 17 -> 11
- net +5V: track 130.7 -> 127.4 mm
- net /CAN_CS: track 19.5 -> 22.8 mm
- net /WHEEL_R: track 22.0 -> 23.3 mm
- net /SENSOR_1: track 33.3 -> 34.3 mm
- net /SENSOR_2: track 27.7 -> 28.7 mm
- net /FAN_SIG: track 29.3 -> 30.2 mm
- net /BRAKE_SIG: track 24.7 -> 25.5 mm
- net /WHEEL_L: track 45.1 -> 46.0 mm
- net /DAMPER_L: track 29.2 -> 30.1 mm
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
Commit message: minor layout update
Parts:
- C1: moved to B.Cu
- R1: moved to F.Cu
- moved R1 12.2 mm to (125.6, 90.9), turned to 90 degrees
- moved C1 10.6 mm to (115.7, 97.9), turned to 270 degrees
- moved Q1 2.82 mm to (131.3, 90.0), turned to 0 degrees
Connections:
- U1 pad 13: (no net) -> /BRAKE_SIG
- U1 pad 2: /BRAKE_SIG -> (no net)
Routing:
- net GND: track 4.53 -> 0.00 mm, vias 11 -> 21
- net /FAN_SIG: track 30.2 -> 28.7 mm
- net +5V: track 127.4 -> 126.0 mm, vias 2 -> 3
- net /BRAKE_SIG: track 25.5 -> 24.7 mm, vias 1 -> 0

Commit message: gerber files
Parts:
- added G***: LOGO, AERO_CUSTOM:AERO_Logo_10x4mm, F.Cu at (156.8, 109.2)
