File: DaqBoard/KiCad/_autosave-DaqBoard.kicad_pcb (KiCad board)
At the start: 2 copper layers, 61 x 41.3 mm, 25 parts, among them J1 RJ45, J2 Conn_01x02, J3 Conn_02x03_Odd_Even, J4 RJ45, J5 Conn_01x23, Q1 PSMN5R2-60YL, Q2 PSMN5R2-60YL, U1 ATmega328P-AU, U2 R-785.0-1.0, U3 MCP2515-xSO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

Commit message: gerber files
Parts:
- added G***: LOGO, AERO_CUSTOM:AERO_Logo_10x4mm, F.Cu at (156.8, 109.2)
