File: Dash/KiCad/Dash_Left/Dash_Left.kicad_pcb (KiCad board)
At the start: 2 copper layers, 86.4 x 93.3 mm, 32 parts, among them J1 Conn_01x04, J2 Conn_02x03_Odd_Even, J3 Conn_01x02, U1 ATmega328P-AU, U2 R-785.0-1.0, U3 RC1602A, U4 STP16CP05, U5 MCP2515-xSO, U6 MCP2551-I-SN, Y1 16MHz

Commit message: first layout design
Parts:
- added G***: LOGO, AERO_CUSTOM:AERO_Logo_15x6mm, B.Cu at (176.5, 46.5)
- added R10: 330, Resistor_SMD:R_0603_1608Metric_Pad0.98x0.95mm_HandSolder, F.Cu at (149.1, 96.9)
- added R11: 330, Resistor_SMD:R_0603_1608Metric_Pad0.98x0.95mm_HandSolder, F.Cu at (147.3, 96.9)
- added R12: 330, Resistor_SMD:R_0603_1608Metric_Pad0.98x0.95mm_HandSolder, F.Cu at (138.2, 96.9)
- added R13: 330, Resistor_SMD:R_0603_1608Metric_Pad0.98x0.95mm_HandSolder, F.Cu at (136.5, 96.9)
- added R14: 330, Resistor_SMD:R_0603_1608Metric_Pad0.98x0.95mm_HandSolder, F.Cu at (134.7, 97.0)
- added R15: 330, Resistor_SMD:R_0603_1608Metric_Pad0.98x0.95mm_HandSolder, F.Cu at (126.0, 97.1)
- added R16: 330, Resistor_SMD:R_0603_1608Metric_Pad0.98x0.95mm_HandSolder, F.Cu at (124.3, 97.0)
- added R17: 330, Resistor_SMD:R_0603_1608Metric_Pad0.98x0.95mm_HandSolder, F.Cu at (122.6, 97.0)
- added R6: 330, Resistor_SMD:R_0603_1608Metric_Pad0.98x0.95mm_HandSolder, F.Cu at (167.3, 97.0)
- added R7: 330, Resistor_SMD:R_0603_1608Metric_Pad0.98x0.95mm_HandSolder, F.Cu at (165.5, 97.0)
- added R8: 330, Resistor_SMD:R_0603_1608Metric_Pad0.98x0.95mm_HandSolder, F.Cu at (163.6, 97.0)
- added R9: 330, Resistor_SMD:R_0603_1608Metric_Pad0.98x0.95mm_HandSolder, F.Cu at (150.8, 96.9)
- C3, C4, C5, C7, F1, Y1: moved to B.Cu
- moved RV1 55.8 mm to (165.1, 81.1), turned to 90 degrees
- moved J2 49.9 mm to (117.3, 111.5), turned to 90 degrees
- moved C6 24.8 mm to (139.4, 111.2), turned to 180 degrees
- moved C4 24.7 mm to (151.8, 80.8)
- moved J3 23.5 mm to (118.4, 104.1)
- moved C7 22.4 mm to (158.5, 111.4), turned to 90 degrees
- moved R3 21.1 mm to (142.9, 111.2)
- moved Y1 18.2 mm to (156.2, 104.4), turned to 90 degrees
- moved C5 16.7 mm to (177.5, 110.0), turned to 0 degrees
- moved U5 14.1 mm to (156.5, 107.7)
- moved U6 13.7 mm to (169.9, 103.7)
- moved R5 11.7 mm to (177.2, 103.0)
- moved R2 11.0 mm to (120.1, 108.1), turned to 180 degrees
- moved C2 10.1 mm to (136.7, 109.1), turned to 270 degrees
- moved R4 8.48 mm to (149.0, 112.5), turned to 90 degrees
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Connections:
- D2 pad 1: /TEMP_IND1R -> Net-(D2-Pad1)
- D2 pad 2: /TEMP_IND1G -> Net-(D2-Pad2)
- D2 pad 3: /TEMP_IND1B -> Net-(D2-Pad3)
- D3 pad 1: /TEMP_IND2R -> Net-(D3-Pad1)
- D3 pad 2: /TEMP_IND2G -> Net-(D3-Pad2)
- D3 pad 3: /TEMP_IND2B -> Net-(D3-Pad3)
- D4 pad 1: /TEMP_IND3R -> Net-(D4-Pad1)
- D4 pad 2: /TEMP_IND3G -> Net-(D4-Pad2)
- D4 pad 3: /TEMP_IND3B -> Net-(D4-Pad3)
- D5 pad 1: /BATT_R -> Net-(D5-Pad1)
- D5 pad 2: /BATT_G -> Net-(D5-Pad2)
- D5 pad 3: /BATT_B -> Net-(D5-Pad3)
- J1 pad 2: /CANL -> /CAN+
- J1 pad 3: /CANH -> /CAN-
- R5 pad 1: /CANH -> /CAN+
- R5 pad 2: /CANL -> /CAN-
- U6 pad 6: /CANL -> /CAN-
- U6 pad 7: /CANH -> /CAN+
Routing:
- net +5V: track 0.00 -> 208.3 mm, vias 0 -> 2
- net /SCK: track 0.00 -> 46.6 mm, vias 0 -> 2
- net /MOSI: track 0.00 -> 44.2 mm, vias 0 -> 2
- net /MISO: track 0.00 -> 41.0 mm, vias 0 -> 2
- net /CAN_CS: track 0.00 -> 28.6 mm, vias 0 -> 2
- net /CAN_INT: track 0.00 -> 27.6 mm, vias 0 -> 2
- net /LCD_RS: track 0.00 -> 26.8 mm, vias 0 -> 1
- net /TEMP_IND1R: track 0.00 -> 26.6 mm
- net /LCD_D7: track 0.00 -> 24.6 mm, vias 0 -> 1
- net /TEMP_IND1G: track 0.00 -> 24.5 mm
- net /LED_LE: track 0.00 -> 24.2 mm, vias 0 -> 2
- net Net-(RV1-Pad2): track 0.00 -> 23.5 mm
- net /LCD_EN: track 0.00 -> 23.2 mm, vias 0 -> 1
- net /LED_SDI: track 0.00 -> 23.1 mm, vias 0 -> 2
- net /LCD_D6: track 0.00 -> 22.6 mm, vias 0 -> 1
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- added copper zone on B.Cu, net GND
- added copper zone on F.Cu, net GND
Other:
- board size 86.4 x 93.3 mm -> 86.4 x 76.2 mm
- board text added: "DASH LEFT G.SPEARING 21.012"

Commit message: update PCB Layout
Routing:
- net /CAN+: track 12.4 -> 14.1 mm
