File: Dash/KiCad/Dash_Left/Dash_Left.sch (KiCad schematic (older format))
At the start: 25 parts

Commit message: first layout design
Parts:
- removed SW?: SW_Push, symbol Switch:SW_Push
- added J3: Conn_01x02, Connector_JST:JST_XH_S2B-XH-A_1x02_P2.50mm_Horizontal, symbol Connector_Generic:Conn_01x02
- added R10, R11, R12, R13, R14, R15, R16, R17, R6, R7, R8, R9: 330, Resistor_SMD:R_0603_1608Metric_Pad0.98x0.95mm_HandSolder, symbol Device:R
- C1, C2, C3, C4, C5, C6: renamed from C?; footprint (none) -> Capacitor_SMD:C_0603_1608Metric_Pad1.08x0.95mm_HandSolder
- D1: renamed from D?; footprint (none) -> LED_SMD:LED_0603_1608Metric_Pad1.05x0.95mm_HandSolder
- D2, D3, D4, D5: renamed from D?; footprint (none) -> LED_THT:LED_D5.0mm-4_RGB
- F1: renamed from F?; footprint (none) -> Fuse:Fuse_1812_4532Metric_Pad1.30x3.40mm_HandSolder
- H1, H2: renamed from H?; footprint (none) -> MountingHole:MountingHole_3.2mm_M3
- J1: renamed from J?; footprint (none) -> Connector_JST:JST_XH_S4B-XH-A_1x04_P2.50mm_Horizontal
- J2: renamed from J?; footprint (none) -> Connector_PinSocket_2.54mm:PinSocket_2x03_P2.54mm_Vertical
- R1, R2, R3: renamed from R?; footprint (none) -> Resistor_SMD:R_0603_1608Metric_Pad0.98x0.95mm_HandSolder
- RV1: renamed from RV?; footprint (none) -> Potentiometer_THT:Potentiometer_Bourns_3386P_Vertical
- U4: renamed from U?; footprint (none) -> Package_SO:TSSOP-24_4.4x7.8mm_P0.65mm
- gave numbers to parts that had none: 3
Connections:
- net BATT_B: now also R17.2; no longer D5.3 (BK)
- net BATT_G: now also R16.2; no longer D5.2 (GK)
- net BATT_R: now also R15.2; no longer D5.1 (RK)
- net GND: now also J3.2 (Pin_2)
- net LCD_BTN: now also J3.1 (Pin_1)
- net TEMP_IND1B: now also R8.2; no longer D2.3 (BK)
- net TEMP_IND1G: now also R7.2; no longer D2.2 (GK)
- net TEMP_IND1R: now also R6.2; no longer D2.1 (RK)
- net TEMP_IND2B: now also R11.2; no longer D3.3 (BK)
- net TEMP_IND2G: now also R10.2; no longer D3.2 (GK)
- net TEMP_IND2R: now also R9.2; no longer D3.1 (RK)
- net TEMP_IND3B: now also R14.2; no longer D4.3 (BK)
- net TEMP_IND3G: now also R13.2; no longer D4.2 (GK)
- net TEMP_IND3R: now also R12.2; no longer D4.1 (RK)
- net CANH renamed CAN-
- net CANL renamed CAN+
- new net: D2.1 (RK), R6.1
- new net: D2.2 (GK), R7.1
- new net: D2.3 (BK), R8.1
- new net: D3.1 (RK), R9.1
- new net: D3.2 (GK), R10.1
- new net: D3.3 (BK), R11.1
- new net: D4.1 (RK), R12.1
- new net: D4.2 (GK), R13.1
- new net: D4.3 (BK), R14.1
- new net: D5.1 (RK), R15.1
- new net: D5.2 (GK), R16.1
- new net: D5.3 (BK), R17.1
Other:
- moved on the sheet: D2, D3, D4, D5, R2

Commit message: update PCB Layout
Other:
- note added: "Left Side Dash\n- Temperature LED\n- LCD display output"
Changed lines of the file:
@@
 Text Label 4125 1775 2    50   ~ 0
 CAN+
+Text Notes 7075 6875 0    50   ~ 0
+Left Side Dash\n- Temperature LED\n- LCD display output
 $EndSCHEMATC
