File: Dash/KiCad/Dash_Right/CAN_Interface.sch (KiCad schematic (older format))
At the start: 7 parts

Commit message: initial pcb layout
Parts:
- C5, C6: renamed from C?; footprint (none) -> Capacitor_SMD:C_0603_1608Metric_Pad1.08x0.95mm_HandSolder
- R8, R9: renamed from R?; footprint (none) -> Resistor_SMD:R_0603_1608Metric_Pad0.98x0.95mm_HandSolder
- Y1: renamed from Y?; footprint (none) -> Crystal:Resonator_SMD_muRata_CSTxExxV-3Pin_3.0x1.1mm_HandSoldering
- gave numbers to parts that had none: 2
Changed lines of the file:
@@
 $EndDescr
 $Comp
-L Interface_CAN_LIN:MCP2515-xSO U?
+L Interface_CAN_LIN:MCP2515-xSO U3
 U 1 1 5FFBACF4
 P 4425 4050
-F 0 "U?" H 4900 4950 50  0000 C CNN
+F 0 "U3" H 4900 4950 50  0000 C CNN
 F 1 "MCP2515-xSO" H 4925 4850 50  0000 C CNN
 F 2 "Package_SO:SOIC-18W_7.5x11.6mm_P1.27mm" H 4425 3150 50  0001 C CIN
@@
 $EndComp
 $Comp
-L Interface_CAN_LIN:MCP2551-I-SN U?
+L Interface_CAN_LIN:MCP2551-I-SN U4
 U 1 1 5FFBACF5
 P 6525 3650
-F 0 "U?" H 6950 4150 50  0000 C CNN
+F 0 "U4" H 6950 4150 50  0000 C CNN
 F 1 "MCP2551-I-SN" H 6900 4050 50  0000 C CNN
 F 2 "Package_SO:SOIC-8_3.9x4.9mm_P1.27mm" H 6525 3150 50  0001 C CIN
@@
 $EndComp
 $Comp
-L power:+5V #PWR?
+L power:+5V #PWR0131
 U 1 1 6011BDC8
 P 4425 2775
-F 0 "#PWR?" H 4425 2625 50  0001 C CNN
+F 0 "#PWR0131" H 4425 2625 50  0001 C CNN
 F 1 "+5V" H 4440 2948 50  0000 C CNN
 F 2 "" H 4425 2775 50  0001 C CNN
@@
 $EndComp
 $Comp
-L power:GND #PWR?
+L power:GND #PWR0132
 U 1 1 6011BDC9
 P 4425 4850
-F 0 "#PWR?" H 4425 4600 50  0001 C CNN
+F 0 "#PWR0132" H 4425 4600 50  0001 C CNN
 F 1 "GND" H 4430 4677 50  0000 C CNN
 F 2 "" H 4425 4850 50  0001 C CNN
@@
 $EndComp
 $Comp
-L power:+5V #PWR?
+L power:+5V #PWR0133
 U 1 1 6011BDCA
 P 5450 4650
-F 0 "#PWR?" H 5450 4500 50  0001 C CNN
+F 0 "#PWR0133" H 5450 4500 50  0001 C CNN
 F 1 "+5V" H 5465 4823 50  0000 C CNN
 F 2 "" H 5450 4650 50  0001 C CNN
@@
 $EndComp
 $Comp
-L Device:C C?
+L Device:C C5
 U 1 1 6011BDCB
 P 3950 2925
-F 0 "C?" H 4065 2971 50  0000 L CNN
+F 0 "C5" H 4065 2971 50  0000 L CNN
 F 1 "0.1u" H 4065 2880 50  0000 L CNN
-F 2 "" H 3988 2775 50  0001 C CNN
+F 2 "Capacitor_SMD:C_0603_1608Metric_Pad1.08x0.95mm_HandSolder" H 3988 2775 50  0001 C CNN
 F 3 "~" H 3950 2925 50  0001 C CNN
 	1    3950 2925
@@
 $EndComp
 $Comp
-L power:GND #PWR?
+L power:GND #PWR0134
 U 1 1 5FFBAD03
 P 3950 3075
-F 0 "#PWR?" H 3950 2825 50  0001 C CNN
+F 0 "#PWR0134" H 3950 2825 50  0001 C CNN
 F 1 "GND" H 3955 2902 50  0000 C CNN
 F 2 "" H 3950 3075 50  0001 C CNN
@@
 Connection ~ 4425 2775
 $Comp
-L Device:R R?
+L Device:R R8
 U 1 1 5FFBAD04
 P 5250 4650
-F 0 "R?" V 5150 4650 50  0000 C CNN
+F 0 "R8" V 5150 4650 50  0000 C CNN
 F 1 "10K" V 5250 4650 50  0000 C CNN
-F 2 "" V 5180 4650 50  0001 C CNN
+F 2 "Resistor_SMD:R_0603_1608Metric_Pad0.98x0.95mm_HandSolder" V 5180 4650 50  0001 C CNN
 F 3 "~" H 5250 4650 50  0001 C CNN
 	1    5250 4650
@@
 	5375 4050 5025 4050
 $Comp
-L power:+5V #PWR?
+L power:+5V #PWR0135
 U 1 1 5FFBAD05
 P 6525 2775
-F 0 "#PWR?" H 6525 2625 50  0001 C CNN
+F 0 "#PWR0135" H 6525 2625 50  0001 C CNN
 F 1 "+5V" H 6540 2948 50  0000 C CNN
 F 2 "" H 6525 2775 50  0001 C CNN
@@
 $EndComp
 $Comp
-L Device:C C?
+L Device:C C6
 U 1 1 60014BBC
 P 6050 2925
-F 0 "C?" H 6165 2971 50  0000 L CNN
+F 0 "C6" H 6165 2971 50  0000 L CNN
 F 1 "0.1u" H 6165 2880 50  0000 L CNN
-F 2 "" H 6088 2775 50  0001 C CNN
+F 2 "Capacitor_SMD:C_0603_1608Metric_Pad1.08x0.95mm_HandSolder" H 6088 2775 50  0001 C CNN
 F 3 "~" H 6050 2925 50  0001 C CNN
 	1    6050 2925
@@
 $EndComp
 $Comp
-L power:GND #PWR?
+L power:GND #PWR0136
 U 1 1 6011BDCF
 P 6050 3075
-F 0 "#PWR?" H 6050 2825 50  0001 C CNN
+F 0 "#PWR0136" H 6050 2825 50  0001 C CNN
 F 1 "GND" H 6055 2902 50  0000 C CNN
 F 2 "" H 6050 3075 50  0001 C CNN
@@
 Connection ~ 6525 2775
 $Comp
-L power:GND #PWR?
+L power:GND #PWR0137
 U 1 1 600190E5
 P 6525 4050
-F 0 "#PWR?" H 6525 3800 50  0001 C CNN
+F 0 "#PWR0137" H 6525 3800 50  0001 C CNN
 F 1 "GND" H 6530 3877 50  0000 C CNN
 F 2 "" H 6525 4050 50  0001 C CNN
@@
 	3700 4625 3600 4625
 $Comp
-L power:GND #PWR?
+L power:GND #PWR0138
 U 1 1 6011BDD8
 P 3450 4825
-F 0 "#PWR?" H 3450 4575 50  0001 C CNN
+F 0 "#PWR0138" H 3450 4575 50  0001 C CNN
 F 1 "GND" H 3455 4652 50  0000 C CNN
 F 2 "" H 3450 4825 50  0001 C CNN
@@
 $EndComp
 $Comp
-L Device:R R?
+L Device:R R9
 U 1 1 6011BDD0
 P 7600 3650
-F 0 "R?" H 7670 3696 50  0000 L CNN
+F 0 "R9" H 7670 3696 50  0000 L CNN
 F 1 "120" V 7600 3575 50  0000 L CNN
-F 2 "" V 7530 3650 50  0001 C CNN
+F 2 "Resistor_SMD:R_0603_1608Metric_Pad0.98x0.95mm_HandSolder" V 7530 3650 50  0001 C CNN
 F 3 "~" H 7600 3650 50  0001 C CNN
 	1    7600 3650
@@
 	3600 3450 3825 3450
 $Comp
-L Device:Resonator Y?
+L Device:Resonator Y1
 U 1 1 6011BDC0
 P 3450 4625
-F 0 "Y?" H 3450 4873 50  0000 C CNN
+F 0 "Y1" H 3450 4873 50  0000 C CNN
 F 1 "16MHz" H 3450 4782 50  0000 C CNN
-F 2 "" H 3425 4625 50  0001 C CNN
+F 2 "Crystal:Resonator_SMD_muRata_CSTxExxV-3Pin_3.0x1.1mm_HandSoldering" H 3425 4625 50  0001 C CNN
 F 3 "~" H 3425 4625 50  0001 C CNN
 	1    3450 4625

Commit message: first layout design
Changed lines of the file:
@@
 Text Label 5125 3550 0    50   ~ 0
 TXCAN
-Text Label 5375 4050 2    50   ~ 0
-CAN_INT
 Wire Wire Line
-	5375 4050 5025 4050
+	5200 4050 5025 4050
 $Comp
 L power:+5V #PWR0135
@@
 Wire Wire Line
 	7600 3500 7875 3500
+Text HLabel 5200 4050 2    50   Input ~ 0
+CAN_INT
 $EndSCHEMATC
