File: Dash/KiCad/Dash_Right/Dash_Right.sch (KiCad schematic (older format))
At the start: 30 parts

Commit message: initial pcb layout
Parts:
- removed J?: Conn_01x02, symbol Connector_Generic:Conn_01x02
- removed Q?: MMBT5551L, Package_TO_SOT_SMD:SOT-23, symbol Transistor_BJT:MMBT5551L
- removed SW? (x2): SW_SPST, symbol Switch:SW_SPST
- added Q1: PSMN5R2-60YL, Package_TO_SOT_SMD:LFPAK56, symbol Transistor_FET:PSMN5R2-60YL
- added SW1, SW2: SW_SPDT, AERO_CUSTOM:Toggle_Switch_100SP1T1B4M2QE, symbol Switch:SW_SPDT
- C1, C2, C3, C4: renamed from C?; footprint (none) -> Capacitor_SMD:C_0603_1608Metric_Pad1.08x0.95mm_HandSolder
- D1: renamed from D?; footprint (none) -> Fuse:Fuse_0603_1608Metric_Pad1.05x0.95mm_HandSolder
- D2, D3, D4: renamed from D?; footprint (none) -> LED_THT:LED_D3.0mm
- F1: renamed from F?; footprint (none) -> Fuse:Fuse_1812_4532Metric_Pad1.30x3.40mm_HandSolder
- H1, H2: renamed from H?; footprint (none) -> MountingHole:MountingHole_3.2mm_M3
- J1, J6: renamed from J?; footprint (none) -> Connector_JST:JST_XH_S4B-XH-A_1x04_P2.50mm_Horizontal
- J2, J3: renamed from J?; footprint (none) -> Connector_JST:JST_XH_S3B-XH-A_1x03_P2.50mm_Horizontal
- J5: renamed from J?; footprint (none) -> Connector_PinHeader_2.54mm:PinHeader_2x03_P2.54mm_Vertical
- J7: renamed from J?; footprint (none) -> AERO_CUSTOM:TE_1-776262-1_14pin_Vertical
- R1, R2, R3, R5, R6, R7: renamed from R?; footprint (none) -> Resistor_SMD:R_0603_1608Metric_Pad0.98x0.95mm_HandSolder
- R4: renamed from R?; value 1K -> 10K; footprint (none) -> Resistor_SMD:R_0603_1608Metric_Pad0.98x0.95mm_HandSolder
- gave numbers to parts that had none: 2
Connections:
- net COOLING: now also SW1.1 (A)
- net DIRECTION: now also SW2.1 (A)
- net GND: now also R4.1, Q1.1 (S), Q1.2 (S), Q1.3 (S), SW1.2 (B), SW2.2 (B)
- net RTD_IND: now also R4.2, Q1.4 (G)
- net SENSOR_1: no longer J7.10 (Pin_10)
- new net RTD_IND_OUT: J7.10 (Pin_10), Q1.5 (D)
Other:
- moved on the sheet: R2, R4

Commit message: first layout design
Connections:
- net +12V: now also J6.1 (Pin_1), J7.14 (Pin_14), J7.9 (Pin_9); no longer J6.4 (Pin_4), J7.1 (Pin_1), J7.2 (Pin_2)
- net +5V: now also J7.4 (Pin_4), J7.5 (Pin_5); no longer J7.7 (Pin_7), J7.9 (Pin_9)
- net BMS_LED: now also U1.2 (PD4); no longer U1.11 (PD7)
- net COOLING: now also U1.26 (PC3); no longer U1.25 (PC2)
- net DIRECTION: now also U1.25 (PC2); no longer U1.26 (PC3)
- net GND: now also J6.4 (Pin_4), J7.10 (Pin_10); no longer J6.1 (Pin_1), J7.14 (Pin_14)
- net IMD_LED: now also U1.10 (PD6); no longer U1.2 (PD4)
- net RTD_BTN: now also J1.3 (Pin_3), U1.12 (PB0); no longer J1.2 (Pin_2), U1.13 (PB1)
- net RTD_IND: now also U1.14 (PB2); no longer U1.12 (PB0)
- net RTD_IND_OUT: now also J7.1 (Pin_1); no longer J7.10 (Pin_10)
- net RTD_LED: now also J1.2 (Pin_2), U1.13 (PB1); no longer J1.3 (Pin_3), U1.14 (PB2)
- net TMS_LED: now also U1.11 (PD7); no longer U1.10 (PD6)
- net CANH renamed CAN-
- net CAN-: now also J7.7 (Pin_7); no longer J7.4 (Pin_4)
- net CANL renamed CAN+
- net CAN+: now also J7.2 (Pin_2); no longer J7.5 (Pin_5)
Changed lines of the file:
@@
 F5 "SCK" I L 5000 5475 50
 F6 "CANH" B R 5925 5225 50
-F7 "CANL" B R 5925 5400 50
+F7 "CANL" B R 5925 5325 50
+F8 "CAN_INT" I R 5925 5450 50
 $EndSheet
 Text Label 4575 5275 0    50   ~ 0
@@
 $EndComp
 $Comp
-L Connector_Generic:Conn_01x14 J7
-U 1 1 60146BEB
-P 10550 5350
-F 0 "J7" H 10630 5342 50  0000 L CNN
-F 1 "Conn_01x14" H 10630 5251 50  0000 L CNN
-F 2 "AERO_CUSTOM:TE_1-776262-1_14pin_Vertical" H 10550 5350 50  0001 C CNN
-F 3 "~" H 10550 5350 50  0001 C CNN
-	1    10550 5350
-	1    0    0    -1
-$EndComp
-$Comp
 L power:+12V #PWR0111
 U 1 1 60147573
-P 10025 4750
-F 0 "#PWR0111" H 10025 4600 50  0001 C CNN
-F 1 "+12V" H 10040 4923 50  0000 C CNN
-F 2 "" H 10025 4750 50  0001 C CNN
-F 3 "" H 10025 4750 50  0001 C CNN
-	1    10025 4750
-	1    0    0    -1
-$EndComp
-Wire Wire Line
-	10025 4750 10350 4750
-Wire Wire Line
-	10025 4750 10025 4850
-Wire Wire Line
-	10025 4850 10350 4850
-Connection ~ 10025 4750
-Text Label 10125 4950 0    50   ~ 0
-CANH
-Wire Wire Line
-	10125 4950 10350 4950
-Wire Wire Line
-	10350 5050 10125 5050
-Wire Wire Line
-	10125 5050 10125 4950
-Text Label 10125 5150 0    50   ~ 0
-CANL
-Wire Wire Line
-	10125 5150 10350 5150
-Wire Wire Line
-	10350 5250 10125 5250
-Wire Wire Line
-	10125 5250 10125 5150
+P 9600 5550
+F 0 "#PWR0111" H 9600 5400 50  0001 C CNN
+F 1 "+12V" H 9615 5723 50  0000 C CNN
+F 2 "" H 9600 5550 50  0001 C CNN
+F 3 "" H 9600 5550 50  0001 C CNN
+	1    9600 5550
+	1    0    0    -1
+$EndComp
+Wire Wire Line
+	9850 5250 10350 5250
+Wire Wire Line
+	9850 5350 10350 5350
 $Comp
 L power:+5V #PWR0112
 U 1 1 601511B0
-P 10025 5350
-F 0 "#PWR0112" H 10025 5200 50  0001 C CNN
-F 1 "+5V" H 10040 5523 50  0000 C CNN
-F 2 "" H 10025 5350 50  0001 C CNN
-F 3 "" H 10025 5350 50  0001 C CNN
-	1    10025 5350
-	1    0    0    -1
-$EndComp
-Wire Wire Line
-	10025 5350 10350 5350
-Wire Wire Line
-	10350 5450 10025 5450
-Wire Wire Line
-	10025 5450 10025 5350
-Connection ~ 10025 5350
-Wire Wire Line
-	10350 5550 10025 5550
-Wire Wire Line
-	10025 5550 10025 5450
-Connection ~ 10025 5450
-Text Label 9850 5650 0    50   ~ 0
+P 9775 5050
+F 0 "#PWR0112" H 9775 4900 50  0001 C CNN
+F 1 "+5V" H 9790 5223 50  0000 C CNN
+F 2 "" H 9775 5050 50  0001 C CNN
+F 3 "" H 9775 5050 50  0001 C CNN
+	1    9775 5050
+	1    0    0    -1
+$EndComp
+Connection ~ 9775 5050
+Text Label 9850 4750 0    50   ~ 0
 RTD_IND_OUT
 Wire Wire Line
-	9850 5650 10350 5650
+	9850 4750 10350 4750
 $Comp
 L power:GND #PWR0113
 U 1 1 601557A0
-P 10025 6050
-F 0 "#PWR0113" H 10025 5800 50  0001 C CNN
-F 1 "GND" H 10030 5877 50  0000 C CNN
-F 2 "" H 10025 6050 50  0001 C CNN
-F 3 "" H 10025 6050 50  0001 C CNN
-	1    10025 6050
-	1    0    0    -1
-$EndComp
-Wire Wire Line
-	10025 6050 10350 6050
-Wire Wire Line
-	10350 5950 10025 5950
-Wire Wire Line
-	10025 5950 10025 6050
-Connection ~ 10025 6050
-Wire Wire Line
-	10350 5850 10025 5850
-Wire Wire Line
-	10025 5850 10025 5950
-Connection ~ 10025 5950
+P 9800 5950
+F 0 "#PWR0113" H 9800 5700 50  0001 C CNN
+F 1 "GND" H 9805 5777 50  0000 C CNN
+F 2 "" H 9800 5950 50  0001 C CNN
+F 3 "" H 9800 5950 50  0001 C CNN
+	1    9800 5950
+	1    0    0    -1
+$EndComp
+Wire Wire Line
+	9800 5950 10350 5950
+Wire Wire Line
+	10350 5850 9800 5850
+Wire Wire Line
+	9800 5850 9800 5950
+Connection ~ 9800 5950
+Wire Wire Line
+	9800 5750 9800 5850
+Connection ~ 9800 5850
 Text Label 3200 4575 2    50   ~ 0
 SENSOR_1
@@
 Wire Wire Line
 	3200 4675 2775 4675
+Text Label 3150 2775 2    50   ~ 0
+RTD_IND
+Wire Wire Line
+	3150 2575 2775 2575
 Text Label 3150 2575 2    50   ~ 0
-RTD_IND
-Wire Wire Line
-	3150 2575 2775 2575
-Text Label 3150 2675 2    50   ~ 0
 RTD_BTN
 Wire Wire Line
@@
 Wire Wire Line
 	3150 3575 2775 3575
+Text Label 3200 3775 2    50   ~ 0
+COOLING
+Wire Wire Line
+	3150 3675 2775 3675
 Text Label 3150 3675 2    50   ~ 0
-COOLING
-Wire Wire Line
-	3150 3675 2775 3675
-Text Label 3200 3775 2    50   ~ 0
 DIRECTION
 Wire Wire Line
@@
 Wire Wire Line
 	4600 1725 4250 1725
+Text Label 4625 1825 2    50   ~ 0
+RTD_BTN
+Wire Wire Line
+	4625 1925 4250 1925
 Text Label 4625 1925 2    50   ~ 0
-RTD_BTN
-Wire Wire Line
-	4625 1925 4250 1925
-Text Label 4625 1825 2    50   ~ 0
 RTD_LED
 Wire Wire Line
 	4625 1825 4250 1825
-Text Label 3150 2775 2    50   ~ 0
+Text Label 3150 2675 2    50   ~ 0
 RTD_LED
 Wire Wire Line
@@
 	1    0    0    1
 $EndComp
+Text Label 3200 4875 2    50   ~ 0
+IMD_LED
+Text Label 3200 4975 2    50   ~ 0
+TMS_LED
+Wire Wire Line
+	3200 4875 2775 4875
 Text Label 3200 4675 2    50   ~ 0
-IMD_LED
-Text Label 3200 4875 2    50   ~ 0
-TMS_LED
-Wire Wire Line
-	3200 4875 2775 4875
-Text Label 3200 4975 2    50   ~ 0
 BMS_LED
 Wire Wire Line
@@
 	6250 2775 6250 1275
 Wire Wire Line
-	10025 5850 10025 5750
-Wire Wire Line
-	10025 5750 10350 5750
-Connection ~ 10025 5850
+	9800 5750 9800 5650
+Wire Wire Line
+	9800 5650 10350 5650
+Connection ~ 9800 5750
 Text Label 6200 5225 2    50   ~ 0
-CANH
-Text Label 6200 5400 2    50   ~ 0
-CANL
-Wire Wire Line
-	6200 5400 5925 5400
+CAN+
+Text Label 6200 5325 2    50   ~ 0
+CAN-
+Wire Wire Line
+	6200 5325 5925 5325
 Wire Wire Line
 	6200 5225 5925 5225
@@
 BOARD \nCONNECTOR
 Wire Wire Line
-	8750 1700 8425 1700
+	8825 2000 8425 2000
 $Comp
 L power:GND #PWR0129
 U 1 1 5FFC2823
-P 8750 2000
-F 0 "#PWR0129" H 8750 1750 50  0001 C CNN
-F 1 "GND" H 8755 1827 50  0000 C CNN
-F 2 "" H 8750 2000 50  0001 C CNN
-F 3 "" H 8750 2000 50  0001 C CNN
-	1    8750 2000
-	1    0    0    -1
-$EndComp
-Wire Wire Line
-	8750 2000 8425 2000
-Text Label 8750 1800 2    50   ~ 0
-CANH
-Wire Wire Line
-	8750 1800 8425 1800
-Text Label 8750 1900 2    50   ~ 0
-CANL
-Wire Wire Line
-	8750 1900 8425 1900
-Wire Notes Line
-	8025 1225 8925 1225
-Wire Notes Line
-	8925 1225 8925 2225
-Wire Notes Line
-	8925 2225 8025 2225
-Wire Notes Line
-	8025 2225 8025 1225
-$Comp
-L power:+12V #PWR0130
-U 1 1 5FFDDB49
 P 8750 1700
-F 0 "#PWR0130" H 8750 1550 50  0001 C CNN
-F 1 "+12V" H 8765 1873 50  0000 C CNN
+F 0 "#PWR0129" H 8750 1450 50  0001 C CNN
+F 1 "GND" H 8800 1750 50  0000 C CNN
 F 2 "" H 8750 1700 50  0001 C CNN
 F 3 "" H 8750 1700 50  0001 C CNN
 	1    8750 1700
+	1    0    0    -1
+$EndComp
+Wire Wire Line
+	8750 1700 8425 1700
+Wire Wire Line
+	8650 1800 8425 1800
+Wire Wire Line
+	8650 1900 8425 1900
+Wire Notes Line
+	8025 1225 8925 1225
+Wire Notes Line
+	8925 1225 8925 2225
+Wire Notes Line
+	8925 2225 8025 2225
+Wire Notes Line
+	8025 2225 8025 1225
+$Comp
+L power:+12V #PWR0130
+U 1 1 5FFDDB49
+P 8825 2000
+F 0 "#PWR0130" H 8825 1850 50  0001 C CNN
+F 1 "+12V" H 8775 1950 50  0000 C CNN
+F 2 "" H 8825 2000 50  0001 C CNN
+F 3 "" H 8825 2000 50  0001 C CNN
+	1    8825 2000
 	1    0    0    -1
 $EndComp
@@
 Wire Wire Line
 	6000 3925 6000 3975
+Wire Wire Line
+	9850 4950 10350 4950
+Wire Wire Line
+	9850 4850 10350 4850
+Wire Wire Line
+	9775 5050 10350 5050
+Wire Wire Line
+	9600 5550 10350 5550
+Wire Wire Line
+	9775 5050 9775 5150
+Wire Wire Line
+	9775 5450 10350 5450
+$Comp
+L power:+5V #PWR0116
+U 1 1 60108628
+P 9775 5450
+F 0 "#PWR0116" H 9775 5300 50  0001 C CNN
+F 1 "+5V" H 9790 5623 50  0000 C CNN
+F 2 "" H 9775 5450 50  0001 C CNN
+F 3 "" H 9775 5450 50  0001 C CNN
+	1    9775 5450
+	1    0    0    -1
+$EndComp
+Wire Wire Line
+	10350 5750 9800 5750
+$Comp
+L power:+12V #PWR0139
+U 1 1 6011D193
+P 9975 6200
+F 0 "#PWR0139" H 9975 6050 50  0001 C CNN
+F 1 "+12V" H 9990 6373 50  0000 C CNN
+F 2 "" H 9975 6200 50  0001 C CNN
+F 3 "" H 9975 6200 50  0001 C CNN
+	1    9975 6200
+	1    0    0    -1
+$EndComp
+Wire Wire Line
+	10350 5150 9775 5150
+$Comp
+L Connector_Generic:Conn_01x14 J7
+U 1 1 60146BEB
+P 10550 5350
+F 0 "J7" H 10630 5342 50  0000 L CNN
+F 1 "Conn_01x14" H 10630 5251 50  0000 L CNN
+F 2 "AERO_CUSTOM:TE_1-776262-1_14pin_Vertical" H 10550 5350 50  0001 C CNN
+F 3 "~" H 10550 5350 50  0001 C CNN
+	1    10550 5350
+	1    0    0    -1
+$EndComp
+Wire Wire Line
+	10350 6050 10350 6200
+Wire Wire Line
+	10350 6200 9975 6200
+Text Label 6250 5450 2    50   ~ 0
+CAN_INT
+Wire Wire Line
+	6250 5450 5925 5450
+Text Label 9850 4850 0    50   ~ 0
+CAN+
+Text Label 9850 4950 0    50   ~ 0
+CAN-
+Text Label 9850 5250 0    50   ~ 0
+CAN+
+Text Label 9850 5350 0    50   ~ 0
+CAN-
+Text Label 8650 1900 2    50   ~ 0
+CAN+
+Text Label 8650 1800 2    50   ~ 0
+CAN-
 $EndSCHEMATC

Commit message: update PCB Layout
Connections:
- net +12V: now also J7.10 (Pin_10), J7.6 (Pin_6); no longer J7.14 (Pin_14), J7.9 (Pin_9)
- net +5V: now also J7.1 (Pin_1), J7.2 (Pin_2), J7.7 (Pin_7); no longer J7.4 (Pin_4), J7.5 (Pin_5), J7.8 (Pin_8)
- net CAN+: now also J7.4 (Pin_4), J7.9 (Pin_9); no longer J7.2 (Pin_2), J7.6 (Pin_6)
- net CAN-: now also J7.8 (Pin_8); no longer J7.7 (Pin_7)
- net GND: now also J7.14 (Pin_14); no longer J7.10 (Pin_10)
- net RTD_IND_OUT: now also J7.5 (Pin_5); no longer J7.1 (Pin_1)
Other:
- note added: "Right Side Dash\n- Fault Indicators\n- Regen Settings\n- Direction, Cooling switches\n- Precharge\n- Start button"
Changed lines of the file:
@@
 L power:+12V #PWR0111
 U 1 1 60147573
-P 9600 5550
-F 0 "#PWR0111" H 9600 5400 50  0001 C CNN
-F 1 "+12V" H 9615 5723 50  0000 C CNN
-F 2 "" H 9600 5550 50  0001 C CNN
-F 3 "" H 9600 5550 50  0001 C CNN
-	1    9600 5550
-	1    0    0    -1
-$EndComp
-Wire Wire Line
-	9850 5250 10350 5250
-Wire Wire Line
-	9850 5350 10350 5350
+P 9725 5250
+F 0 "#PWR0111" H 9725 5100 50  0001 C CNN
+F 1 "+12V" H 9740 5423 50  0000 C CNN
+F 2 "" H 9725 5250 50  0001 C CNN
+F 3 "" H 9725 5250 50  0001 C CNN
+	1    9725 5250
+	1    0    0    -1
+$EndComp
+Wire Wire Line
+	9850 5550 10350 5550
+Wire Wire Line
+	9850 5450 10350 5450
 $Comp
 L power:+5V #PWR0112
 U 1 1 601511B0
-P 9775 5050
-F 0 "#PWR0112" H 9775 4900 50  0001 C CNN
-F 1 "+5V" H 9790 5223 50  0000 C CNN
-F 2 "" H 9775 5050 50  0001 C CNN
-F 3 "" H 9775 5050 50  0001 C CNN
-	1    9775 5050
-	1    0    0    -1
-$EndComp
-Connection ~ 9775 5050
-Text Label 9850 4750 0    50   ~ 0
+P 9775 4750
+F 0 "#PWR0112" H 9775 4600 50  0001 C CNN
+F 1 "+5V" H 9790 4923 50  0000 C CNN
+F 2 "" H 9775 4750 50  0001 C CNN
+F 3 "" H 9775 4750 50  0001 C CNN
+	1    9775 4750
+	1    0    0    -1
+$EndComp
+Connection ~ 9775 4750
+Text Label 9850 5150 0    50   ~ 0
 RTD_IND_OUT
 Wire Wire Line
-	9850 4750 10350 4750
+	9850 5150 10350 5150
 $Comp
 L power:GND #PWR0113
 U 1 1 601557A0
-P 9800 5950
-F 0 "#PWR0113" H 9800 5700 50  0001 C CNN
-F 1 "GND" H 9805 5777 50  0000 C CNN
-F 2 "" H 9800 5950 50  0001 C CNN
-F 3 "" H 9800 5950 50  0001 C CNN
-	1    9800 5950
-	1    0    0    -1
-$EndComp
-Wire Wire Line
-	9800 5950 10350 5950
-Wire Wire Line
-	10350 5850 9800 5850
+P 9800 6050
+F 0 "#PWR0113" H 9800 5800 50  0001 C CNN
+F 1 "GND" H 9805 5877 50  0000 C CNN
+F 2 "" H 9800 6050 50  0001 C CNN
+F 3 "" H 9800 6050 50  0001 C CNN
+	1    9800 6050
+	1    0    0    -1
+$EndComp
+Wire Wire Line
+	9800 6050 10350 6050
+Wire Wire Line
+	10350 5950 9800 5950
+Wire Wire Line
+	9800 5950 9800 6050
+Connection ~ 9800 6050
 Wire Wire Line
 	9800 5850 9800 5950
 Connection ~ 9800 5950
-Wire Wire Line
-	9800 5750 9800 5850
-Connection ~ 9800 5850
 Text Label 3200 4575 2    50   ~ 0
 SENSOR_1
@@
 	6250 2775 6250 1275
 Wire Wire Line
-	9800 5750 9800 5650
-Wire Wire Line
-	9800 5650 10350 5650
-Connection ~ 9800 5750
+	9800 5850 9800 5750
+Wire Wire Line
+	9800 5750 10350 5750
+Connection ~ 9800 5850
 Text Label 6200 5225 2    50   ~ 0
 CAN+
@@
 	9850 4950 10350 4950
 Wire Wire Line
-	9850 4850 10350 4850
-Wire Wire Line
-	9775 5050 10350 5050
-Wire Wire Line
-	9600 5550 10350 5550
-Wire Wire Line
-	9775 5050 9775 5150
-Wire Wire Line
-	9775 5450 10350 5450
+	9850 5050 10350 5050
+Wire Wire Line
+	9775 4750 10350 4750
+Wire Wire Line
+	9725 5250 10350 5250
+Wire Wire Line
+	9775 4750 9775 4850
+Wire Wire Line
+	9600 5350 10350 5350
 $Comp
 L power:+5V #PWR0116
 U 1 1 60108628
-P 9775 5450
-F 0 "#PWR0116" H 9775 5300 50  0001 C CNN
-F 1 "+5V" H 9790 5623 50  0000 C CNN
-F 2 "" H 9775 5450 50  0001 C CNN
-F 3 "" H 9775 5450 50  0001 C CNN
-	1    9775 5450
-	1    0    0    -1
-$EndComp
-Wire Wire Line
-	10350 5750 9800 5750
+P 9600 5350
+F 0 "#PWR0116" H 9600 5200 50  0001 C CNN
+F 1 "+5V" H 9615 5523 50  0000 C CNN
+F 2 "" H 9600 5350 50  0001 C CNN
+F 3 "" H 9600 5350 50  0001 C CNN
+	1    9600 5350
+	1    0    0    -1
+$EndComp
+Wire Wire Line
+	10350 5850 9800 5850
 $Comp
 L power:+12V #PWR0139
 U 1 1 6011D193
-P 9975 6200
-F 0 "#PWR0139" H 9975 6050 50  0001 C CNN
-F 1 "+12V" H 9990 6373 50  0000 C CNN
-F 2 "" H 9975 6200 50  0001 C CNN
-F 3 "" H 9975 6200 50  0001 C CNN
-	1    9975 6200
-	1    0    0    -1
-$EndComp
-Wire Wire Line
-	10350 5150 9775 5150
+P 9750 5650
+F 0 "#PWR0139" H 9750 5500 50  0001 C CNN
+F 1 "+12V" H 9765 5823 50  0000 C CNN
+F 2 "" H 9750 5650 50  0001 C CNN
+F 3 "" H 9750 5650 50  0001 C CNN
+	1    9750 5650
+	1    0    0    -1
+$EndComp
+Wire Wire Line
+	10350 4850 9775 4850
 $Comp
 L Connector_Generic:Conn_01x14 J7
@@
 $EndComp
 Wire Wire Line
-	10350 6050 10350 6200
-Wire Wire Line
-	10350 6200 9975 6200
+	10350 5650 9750 5650
 Text Label 6250 5450 2    50   ~ 0
 CAN_INT
 Wire Wire Line
 	6250 5450 5925 5450
-Text Label 9850 4850 0    50   ~ 0
+Text Label 9850 5050 0    50   ~ 0
 CAN+
 Text Label 9850 4950 0    50   ~ 0
 CAN-
-Text Label 9850 5250 0    50   ~ 0
+Text Label 9850 5550 0    50   ~ 0
 CAN+
-Text Label 9850 5350 0    50   ~ 0
+Text Label 9850 5450 0    50   ~ 0
 CAN-
 Text Label 8650 1900 2    50   ~ 0
@@
 Text Label 8650 1800 2    50   ~ 0
 CAN-
+Text Notes 7025 7075 0    50   ~ 0
+Right Side Dash\n- Fault Indicators\n- Regen Settings\n- Direction, Cooling switches\n- Precharge\n- Start button
 $EndSCHEMATC

Commit message: Variable Delcarations, Some Functions
Other:
- note added: "Buzzer is +12V"
Changed lines of the file:
@@
 	1    0    0    -1
 $EndComp
-Text Notes 5525 3275 0    50   ~ 0
+Text Notes 6200 3275 0    50   ~ 0
 RTD BUZZER
 $Comp
@@
 Text Notes 7025 7075 0    50   ~ 0
 Right Side Dash\n- Fault Indicators\n- Regen Settings\n- Direction, Cooling switches\n- Precharge\n- Start button
+Text Notes 6200 3350 0    50   ~ 0
+Buzzer is +12V
 $EndSCHEMATC

Commit message: Minor updates
Connections:
- net RTD_BTN: now also U1.1 (PD3); no longer U1.12 (PB0)
- net SENSOR_1: now also U1.12 (PB0); no longer U1.1 (PD3)
Changed lines of the file:
@@
 	9800 5850 9800 5950
 Connection ~ 9800 5950
-Text Label 3200 4575 2    50   ~ 0
+Text Label 3200 2575 2    50   ~ 0
 SENSOR_1
 Wire Wire Line
@@
 RTD_IND
 Wire Wire Line
-	3150 2575 2775 2575
-Text Label 3150 2575 2    50   ~ 0
+	3200 2575 2775 2575
+Text Label 3200 4575 2    50   ~ 0
 RTD_BTN
 Wire Wire Line
