File: Dash/KiCad/Dash_Right/_autosave-Dash_Right.kicad_pcb (KiCad board)
At the start: 2 copper layers, 78.7 x 69.2 mm, 36 parts, among them J1 Conn_01x04, J2 Conn_01x03, J3 Conn_01x03, J5 Conn_02x03_Odd_Even, J6 Conn_01x04, J7 Conn_01x14, Q1 PSMN5R2-60YL, SW1 SW_SPDT, SW2 SW_SPDT, U1 ATmega328P-AU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

Commit message: gerber files
Parts:
- added G***: LOGO, AERO_CUSTOM:AERO_Logo_10x4mm, B.Cu at (184.8, 85.1)
Other:
- rule pad_to_mask_clearance: 0.051 -> 0
