File: FaultLatcher/Kicad/FaultLatcher.sch (KiCad schematic (older format))
At the start: 35 parts, among them J2 Conn_01x14, K1 G5V-2, K2 G5V-2, K3 G5V-2, K4 G5V-2, Q1 2N7002, Q2 2N7002, Q3 2N7002, Q4 2N7002, SW1 SW_Push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

Commit message: update PCB Layout
Parts:
- removed Q1, Q2, Q3: 2N7002, Package_TO_SOT_SMD:SOT-23, symbol Transistor_FET:2N7002
- added D5: LED, LED_SMD:LED_0603_1608Metric_Pad1.05x0.95mm_HandSolder, symbol Device:LED
- added F1: Polyfuse, Fuse:Fuse_1812_4532Metric_Pad1.30x3.40mm_HandSolder, symbol Device:Polyfuse
- added Q1, Q2, Q3: BSS84, Package_TO_SOT_SMD:SOT-23, symbol Transistor_FET:BSS84
- added R7: 330, Fuse:Fuse_0603_1608Metric_Pad1.05x0.95mm_HandSolder, symbol Device:R
- added R8: 4.7k, Resistor_SMD:R_0603_1608Metric_Pad0.98x0.95mm_HandSolder, symbol Device:R
- BMS1: renamed from SW1; footprint (none) -> Connector_JST:JST_PH_B2B-PH-K_1x02_P2.00mm_Vertical
- C1, C2, C3, C4, C5, C6: renamed from C?; footprint (none) -> Capacitor_SMD:C_0603_1608Metric_Pad1.08x0.95mm_HandSolder
- D1, D2, D3, D4: footprint Diode_THT:D_DO-35_SOD27_P7.62mm_Horizontal -> Diode_SMD:D_SOD-123
- IMD1: renamed from SW?; footprint (none) -> Connector_JST:JST_PH_B2B-PH-K_1x02_P2.00mm_Vertical
- J1: renamed from J?; footprint (none) -> Connector_PinHeader_2.54mm:PinHeader_2x03_P2.54mm_Vertical
- J2: footprint (none) -> AERO_CUSTOM:TE_1-776262-1_14pin_Vertical
- R1, R2, R3, R4, R5, R6: renamed from R?; footprint (none) -> Resistor_SMD:R_0603_1608Metric_Pad0.98x0.95mm_HandSolder
- TMS2: renamed from SW3; footprint (none) -> Connector_JST:JST_PH_B2B-PH-K_1x02_P2.00mm_Vertical
- TSM1: renamed from SW2; footprint (none) -> Connector_JST:JST_PH_B2B-PH-K_1x02_P2.00mm_Vertical
- Y1: renamed from Y?; footprint (none) -> AERO_CUSTOM:Resonator_SMD_muRata_CSTxExxV-3Pin_3.0x1.1mm_HandSoldering
- gave numbers to parts that had none: 3
Connections:
- net +12V: now also J2.14 (Pin_14), J2.9 (Pin_9), F1.2; no longer C5.1, J2.2 (Pin_2), J2.6 (Pin_6), R1.1, R2.1, R3.1, U4.1 (IN)
- net +5V: now also Q1.2 (S), Q2.2 (S), Q3.2 (S), R7.2
- net BMS_FAULT: now also J2.5 (Pin_5); no longer J2.10 (Pin_10)
- net BMS_IND: now also U1.11 (PD7), Q1.3 (D); no longer U1.1 (PD3)
- net GND: now also D4.2 (A), J2.1 (Pin_1), J2.2 (Pin_2), R1.1, R2.1, R3.1, D5.1 (K), R8.1; no longer J2.14 (Pin_14), J2.7 (Pin_7)
- net IMD_FAULT: now also J2.3 (Pin_3); no longer J2.13 (Pin_13)
- net IMD_IND: now also U1.1 (PD3), R8.2; no longer U1.11 (PD7)
- net LOOP_IN: now also J2.13 (Pin_13); no longer J2.1 (Pin_1)
- net LOOP_OUT: now also J2.12 (Pin_12); no longer J2.5 (Pin_5)
- net TMS1_FAULT: now also J2.4 (Pin_4); no longer J2.11 (Pin_11), J2.12 (Pin_12)
- net TMS1_IND: now also U1.10 (PD6), Q2.3 (D); no longer U1.2 (PD4)
- net TMS2_FAULT: now also J2.8 (Pin_8)
- net TMS2_IND: now also U1.2 (PD4), Q3.3 (D); no longer U1.10 (PD6)
- net at BMS1.2, D1.2 (A), K1.1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: now also Q1.1 (G)
- net at D2.2 (A), K2.1, K2.8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: now also Q2.1 (G)
- net at D3.2 (A), K3.1, K3.8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: now also Q3.1 (G)
- net at IMD1.2, K4.1, K4.8: now also D4.1 (K), Q4.1 (G)
- net CANH renamed CAN+
- net CAN+: now also J2.10 (Pin_10), J2.6 (Pin_6); no longer J2.3 (Pin_3), J2.8 (Pin_8)
- net CANL renamed CAN-
- net CAN-: now also J2.11 (Pin_11), J2.7 (Pin_7); no longer J2.4 (Pin_4), J2.9 (Pin_9)
- new net: C5.1, F1.1, U4.1 (IN)
- new net: D5.2 (A), R7.1
Other:
- note added: "Fault Latcher\n- Catch / Latch Faults from: \nBMS, IMD, TMS (1 and 2)\n"
- moved on the sheet: C3, C4, C5, C6, J1, J2, R1, R2, R3, R4, R5, R6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
