File: PedalBoard/KiCad/PedalBaord/PedalBaord.kicad_pcb (KiCad board)
At the start: 2 copper layers, 20 parts, among them J1 Conn_02x03_Odd_Even, J2 Conn_01x23, U1 ATmega328P-AU, U2 R-785.0-1.0, U3 MCP2515-xSO, U4 MCP2551-I-SN, Y1 16MHz

Commit message: first layout design
Parts:
- added C7: 0.1u, Capacitor_SMD:C_0603_1608Metric_Pad1.08x0.95mm_HandSolder, F.Cu at (125.7, 80.6)
- added G***: LOGO, AERO_CUSTOM:AERO_Logo_10x4mm, B.Cu at (159.3, 56.8)
- added U5: MCP3008, Package_SO:SOIC-16_3.9x9.9mm_P1.27mm, F.Cu at (125.7, 74.3)
- C2, C5, C6, R4, R5, U4, Y1: moved to B.Cu
- moved C5 11.0 mm to (139.7, 79.1), turned to 90 degrees
- moved U3 10.7 mm to (139.5, 75.6)
- moved D1 9.94 mm to (149.2, 77.5), turned to 180 degrees
- moved C6 9.38 mm to (149.2, 77.5), turned to 180 degrees
- moved C1 8.71 mm to (105.2, 79.4), turned to 180 degrees
- moved R4 8.67 mm to (137.8, 79.1), turned to 90 degrees
- moved Y1 8.26 mm to (137.2, 72.4), turned to 90 degrees
- moved R2 8.00 mm to (117.2, 66.7)
- moved U4 7.70 mm to (147.3, 72.4)
- moved C2 6.74 mm to (114.3, 73.4), turned to 90 degrees
- moved R5 5.43 mm to (143.5, 66.3), turned to 90 degrees
- moved C3 3.91 mm to (153.4, 79.4)
- moved U1 3.66 mm to (113.9, 74.3)
- moved F1 3.55 mm to (154.3, 67.9), turned to 90 degrees
- moved R1 2.59 mm to (113.4, 66.7), turned to 180 degrees
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Connections:
- J2 pad 1: /STEER -> GND
- J2 pad 10: /SENSOR_3 -> /ACC1
- J2 pad 11: /SENSOR_4 -> /STEER
- J2 pad 12: +5V -> /DAMPER_L
- J2 pad 13: +5V -> /CAN+
- J2 pad 14: +5V -> /CAN-
- J2 pad 15: +5V -> +12V
- J2 pad 16: /CANL -> /BRAKE0
- J2 pad 17: /CANL -> /BRAKE1
- J2 pad 18: +12V -> /DAMPER_R
- J2 pad 19: +12V -> /WHEEL_R
- J2 pad 2: /BRAKE0 -> GND
- J2 pad 20: GND -> /WHEEL_L
- J2 pad 21: GND -> /CAN+
- J2 pad 22: GND -> /CAN-
- J2 pad 23: GND -> +12V
- J2 pad 3: /BRAKE1 -> GND
- J2 pad 4: /ACC0 -> GND
- J2 pad 5: /ACC1 -> +5V
- J2 pad 6: /SENSOR_1 -> +5V
- J2 pad 7: /CANH -> +5V
- J2 pad 8: /CANH -> +5V
- J2 pad 9: /SENSOR_2 -> /ACC0
- R1 pad 1: /ACC1 -> /ACC0
- R2 pad 1: /ACC0 -> /ACC1
- R5 pad 1: /CANH -> /CAN+
- R5 pad 2: /CANL -> /CAN-
- U1 pad 1: /SENSOR_1 -> (no net)
- U1 pad 10: /SENSOR_3 -> (no net)
- U1 pad 11: /SENSOR_4 -> (no net)
- U1 pad 13: (no net) -> /ADC_CS
- U1 pad 2: /SENSOR_2 -> (no net)
- U1 pad 24: /BRAKE0 -> /BRAKE1
- U1 pad 25: /BRAKE1 -> /BRAKE0
- U1 pad 26: /ACC0 -> /ACC1
- U1 pad 27: /ACC1 -> /ACC0
- U4 pad 6: /CANL -> /CAN-
- U4 pad 7: /CANH -> /CAN+
Routing:
- net +5V: track 0.00 -> 133.0 mm, vias 0 -> 2
- net /SCK: track 0.00 -> 48.2 mm, vias 0 -> 2
- net /MISO: track 0.00 -> 44.7 mm, vias 0 -> 4
- net /MOSI: track 0.00 -> 40.8 mm, vias 0 -> 3
- net /CAN_INT: track 0.00 -> 26.8 mm, vias 0 -> 2
- net /CAN_CS: track 0.00 -> 25.4 mm, vias 0 -> 2
- net /DAMPER_L: track 0.00 -> 25.1 mm
- net /CAN+: track 0.00 -> 23.0 mm
- net /CAN-: track 0.00 -> 21.7 mm
- net /RESET: track 0.00 -> 21.2 mm
- net /WHEEL_L: track 0.00 -> 21.1 mm
- net /STEER: track 0.00 -> 20.9 mm
- net /ACC1: track 0.00 -> 19.6 mm
- net /WHEEL_R: track 0.00 -> 19.2 mm
- net /DAMPER_R: track 0.00 -> 17.4 mm
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- added copper zone on B.Cu, net +12V
- added copper zone on F.Cu, net +5V
- added copper zone on B.Cu, net GND
- added copper zone on F.Cu, net GND
- added copper zone on B.Cu, net Net-(C3-Pad1)
Other:
- board outline added: 61 x 32.2 mm
- board text added: "PEDAL BOARD G.SPEARING 21.012"

Commit message: update PCB Layout
Routing:
- net /CAN-: track 21.7 -> 23.0 mm
