File: PacMan/KiCad/Packman2020/Packman2020.sch (KiCad schematic (older format))
At the start: 0 parts

Commit message: Minor updates
Parts:
- added C1, C2: 0.1u, Capacitor_SMD:C_0603_1608Metric_Pad1.08x0.95mm_HandSolder, symbol Device:C
- added C3: 1u, Capacitor_SMD:C_0603_1608Metric_Pad1.08x0.95mm_HandSolder, symbol Device:C
- added C4: 10u, Capacitor_SMD:C_0603_1608Metric_Pad1.08x0.95mm_HandSolder, symbol Device:C
- added D5: LED, LED_SMD:LED_0603_1608Metric_Pad1.05x0.95mm_HandSolder, symbol Device:LED
- added D6: 1N4148, Diode_THT:D_DO-35_SOD27_P7.62mm_Horizontal, symbol Diode:1N4148
- added F3: MF-MSMF050, Fuse:Fuse_1812_4532Metric_Pad1.30x3.40mm_HandSolder, symbol Device:Polyfuse
- added H1, H2, H3, H4: MountingHole, MountingHole:MountingHole_3.2mm_M3, symbol Mechanical:MountingHole
- added J10, J11, J12, J9: Conn_01x02, Connector_JST:JST_VH_B2P-VH-B_1x02_P3.96mm_Vertical, symbol Connector_Generic:Conn_01x02
- added J13: Conn_01x14, AERO_CUSTOM:TE_1-776262-1_14pin_Vertical, symbol Connector_Generic:Conn_01x14
- added J5: Conn_02x03_Odd_Even, Connector_PinHeader_2.00mm:PinHeader_2x03_P2.00mm_Vertical, symbol Connector_Generic:Conn_02x03_Odd_Even
- added J6, J7: Conn_01x01, Connector_Hirose:Hirose_DF63R-1P-3.96DSA_1x01_P3.96mm_Vertical, symbol Connector_Generic:Conn_01x01
- added J8: Conn_01x02, Connector_Phoenix_MC_HighVoltage:PhoenixContact_MCV_1,5_2-GF-5.08_1x02_P5.08mm_Vertical_ThreadedFlange_MountHole, symbol Connector_Generic:Conn_01x02
- added Q2: DMN3404L, Package_TO_SOT_SMD:SOT-23, symbol Transistor_FET:DMN3404L
- added R4: 330, Resistor_SMD:R_0603_1608Metric_Pad0.98x0.95mm_HandSolder, symbol Device:R
- added R5: 39k, Resistor_THT:R_Axial_DIN0617_L17.0mm_D6.0mm_P30.48mm_Horizontal, symbol Device:R
- added R6: 10k, Resistor_SMD:R_0603_1608Metric_Pad0.98x0.95mm_HandSolder, symbol Device:R
- added U1: R-785.0-1.0, Converter_DCDC:Converter_DCDC_RECOM_R-78E-0.5_THT, symbol Regulator_Switching:R-785.0-1.0
- added U2: ATmega328P-AU, Package_QFP:TQFP-32_7x7mm_P0.8mm, symbol MCU_Microchip_ATmega:ATmega328P-AU
Connections:
- new net: C2.1, U2.20 (AREF)
- new net: C3.1, F3.1, U1.1 (IN)
- new net: D5.2 (A), R4.1
- new net: J6.1 (Pin_1), R5.1
- new net: J8.1 (Pin_1), R5.2
- new net: J7.1 (Pin_1), J8.2 (Pin_2)
- new net +12V: F3.2, J10.1 (Pin_1), J11.1 (Pin_1), J12.1 (Pin_1), J13.5 (Pin_5), J13.6 (Pin_6), J9.1 (Pin_1)
- new net +5V: C1.1, C4.1, J5.2 (Pin_2), R4.2, U1.3 (OUT), U2.18 (AVCC), U2.4 (VCC), U2.6 (VCC)
- new net CAN+: J13.1 (Pin_1), J13.3 (Pin_3)
- new net CAN-: J13.2 (Pin_2), J13.4 (Pin_4)
- new net CAN_CS: U2.9 (PD5)
- new net CAN_INT: U2.32 (PD2)
- new net CONTACTOR: J13.8 (Pin_8)
- new net FAN_CTRL: Q2.1 (G), R6.1, U2.1 (PD3)
- new net FAN_OUT: D6.1 (K), J10.2 (Pin_2), J11.2 (Pin_2), J12.2 (Pin_2), J9.2 (Pin_2), Q2.3 (D)
- new net GND: C1.2, C2.2, C3.2, C4.2, D5.1 (K), D6.2 (A), J13.13 (Pin_13), J13.14 (Pin_14), J5.6 (Pin_6), Q2.2 (S), R6.2, U1.2 (GND), U2.21 (GND), U2.3 (GND), U2.5 (GND)
- new net MISO: J5.1 (Pin_1), U2.16 (PB4)
- new net MOSI: J5.4 (Pin_4), U2.15 (PB3)
- new net PRECHARGE: J13.7 (Pin_7)
- new net RESET: J5.5 (Pin_5), U2.29 (~RESET~/PC6)
- new net SCK: J5.3 (Pin_3), U2.17 (PB5)
- new net SHUTDOWN_IN: J13.9 (Pin_9)
Other:
- note added: "60V \nINDICATOR\n"
- note added: "HV+\n"
- note added: "HV-\n"
- note added: "PACK FAN\nCONTROL"
