File: PacMan/KiCad/Pacman2020/CAN_Interface.sch (KiCad schematic (older format))
At the start: 7 parts

Commit message: update file names
Parts:
- C5, C6: renamed from C?; footprint (none) -> Capacitor_SMD:C_0603_1608Metric_Pad1.08x0.95mm_HandSolder
- R7, R8: renamed from R?; footprint (none) -> Resistor_SMD:R_0603_1608Metric_Pad0.98x0.95mm_HandSolder
- Y1: renamed from Y?; footprint (none) -> AERO_CUSTOM:Resonator_SMD_muRata_CSTxExxV-3Pin_3.0x1.1mm_HandSoldering
- gave numbers to parts that had none: 2
Changed lines of the file:
@@
 $EndDescr
 $Comp
-L Interface_CAN_LIN:MCP2515-xSO U?
+L Interface_CAN_LIN:MCP2515-xSO U3
 U 1 1 5FFC8CD1
 P 4650 3825
-F 0 "U?" H 5125 4725 50  0000 C CNN
+F 0 "U3" H 5125 4725 50  0000 C CNN
 F 1 "MCP2515-xSO" H 5150 4625 50  0000 C CNN
 F 2 "Package_SO:SOIC-18W_7.5x11.6mm_P1.27mm" H 4650 2925 50  0001 C CIN
@@
 $EndComp
 $Comp
-L Interface_CAN_LIN:MCP2551-I-SN U?
+L Interface_CAN_LIN:MCP2551-I-SN U4
 U 1 1 5FFC8CD2
 P 6750 3425
-F 0 "U?" H 7175 3925 50  0000 C CNN
+F 0 "U4" H 7175 3925 50  0000 C CNN
 F 1 "MCP2551-I-SN" H 7125 3825 50  0000 C CNN
 F 2 "Package_SO:SOIC-8_3.9x4.9mm_P1.27mm" H 6750 2925 50  0001 C CIN
@@
 $EndComp
 $Comp
-L power:+5V #PWR?
+L power:+5V #PWR0118
 U 1 1 5FFBACFF
 P 4650 2550
-F 0 "#PWR?" H 4650 2400 50  0001 C CNN
+F 0 "#PWR0118" H 4650 2400 50  0001 C CNN
 F 1 "+5V" H 4665 2723 50  0000 C CNN
 F 2 "" H 4650 2550 50  0001 C CNN
@@
 $EndComp
 $Comp
-L power:GND #PWR?
+L power:GND #PWR0119
 U 1 1 5FFC8CD8
 P 4650 4625
-F 0 "#PWR?" H 4650 4375 50  0001 C CNN
+F 0 "#PWR0119" H 4650 4375 50  0001 C CNN
 F 1 "GND" H 4655 4452 50  0000 C CNN
 F 2 "" H 4650 4625 50  0001 C CNN
@@
 $EndComp
 $Comp
-L power:+5V #PWR?
+L power:+5V #PWR0120
 U 1 1 5FFC8CD9
 P 5675 4425
-F 0 "#PWR?" H 5675 4275 50  0001 C CNN
+F 0 "#PWR0120" H 5675 4275 50  0001 C CNN
 F 1 "+5V" H 5690 4598 50  0000 C CNN
 F 2 "" H 5675 4425 50  0001 C CNN
@@
 $EndComp
 $Comp
-L Device:C C?
+L Device:C C5
 U 1 1 5FFBAD02
 P 4175 2700
-F 0 "C?" H 4290 2746 50  0000 L CNN
+F 0 "C5" H 4290 2746 50  0000 L CNN
 F 1 "0.1u" H 4290 2655 50  0000 L CNN
-F 2 "" H 4213 2550 50  0001 C CNN
+F 2 "Capacitor_SMD:C_0603_1608Metric_Pad1.08x0.95mm_HandSolder" H 4213 2550 50  0001 C CNN
 F 3 "~" H 4175 2700 50  0001 C CNN
 	1    4175 2700
@@
 $EndComp
 $Comp
-L power:GND #PWR?
+L power:GND #PWR0121
 U 1 1 60083B50
 P 4175 2850
-F 0 "#PWR?" H 4175 2600 50  0001 C CNN
+F 0 "#PWR0121" H 4175 2600 50  0001 C CNN
 F 1 "GND" H 4180 2677 50  0000 C CNN
 F 2 "" H 4175 2850 50  0001 C CNN
@@
 Connection ~ 4650 2550
 $Comp
-L Device:R R?
+L Device:R R7
 U 1 1 5FFC8CDC
 P 5475 4425
-F 0 "R?" V 5375 4425 50  0000 C CNN
+F 0 "R7" V 5375 4425 50  0000 C CNN
 F 1 "10K" V 5475 4425 50  0000 C CNN
-F 2 "" V 5405 4425 50  0001 C CNN
+F 2 "Resistor_SMD:R_0603_1608Metric_Pad0.98x0.95mm_HandSolder" V 5405 4425 50  0001 C CNN
 F 3 "~" H 5475 4425 50  0001 C CNN
 	1    5475 4425
@@
 	3825 3425 4050 3425
 $Comp
-L power:+5V #PWR?
+L power:+5V #PWR0122
 U 1 1 5FFC8CDD
 P 6750 2550
-F 0 "#PWR?" H 6750 2400 50  0001 C CNN
+F 0 "#PWR0122" H 6750 2400 50  0001 C CNN
 F 1 "+5V" H 6765 2723 50  0000 C CNN
 F 2 "" H 6750 2550 50  0001 C CNN
@@
 $EndComp
 $Comp
-L Device:C C?
+L Device:C C6
 U 1 1 60014BBC
 P 6275 2700
-F 0 "C?" H 6390 2746 50  0000 L CNN
+F 0 "C6" H 6390 2746 50  0000 L CNN
 F 1 "0.1u" H 6390 2655 50  0000 L CNN
-F 2 "" H 6313 2550 50  0001 C CNN
+F 2 "Capacitor_SMD:C_0603_1608Metric_Pad1.08x0.95mm_HandSolder" H 6313 2550 50  0001 C CNN
 F 3 "~" H 6275 2700 50  0001 C CNN
 	1    6275 2700
@@
 $EndComp
 $Comp
-L power:GND #PWR?
+L power:GND #PWR0123
 U 1 1 5FFC8CDE
 P 6275 2850
-F 0 "#PWR?" H 6275 2600 50  0001 C CNN
+F 0 "#PWR0123" H 6275 2600 50  0001 C CNN
 F 1 "GND" H 6280 2677 50  0000 C CNN
 F 2 "" H 6275 2850 50  0001 C CNN
@@
 Connection ~ 6750 2550
 $Comp
-L power:GND #PWR?
+L power:GND #PWR0124
 U 1 1 5FFC8CE8
 P 6750 3825
-F 0 "#PWR?" H 6750 3575 50  0001 C CNN
+F 0 "#PWR0124" H 6750 3575 50  0001 C CNN
 F 1 "GND" H 6755 3652 50  0000 C CNN
 F 2 "" H 6750 3825 50  0001 C CNN
@@
 	3925 4400 3825 4400
 $Comp
-L power:GND #PWR?
+L power:GND #PWR0125
 U 1 1 6002416B
 P 3675 4600
-F 0 "#PWR?" H 3675 4350 50  0001 C CNN
+F 0 "#PWR0125" H 3675 4350 50  0001 C CNN
 F 1 "GND" H 3680 4427 50  0000 C CNN
 F 2 "" H 3675 4600 50  0001 C CNN
@@
 $EndComp
 $Comp
-L Device:R R?
+L Device:R R8
 U 1 1 5FFC8CDF
 P 7825 3425
-F 0 "R?" H 7895 3471 50  0000 L CNN
+F 0 "R8" H 7895 3471 50  0000 L CNN
 F 1 "120" V 7825 3350 50  0000 L CNN
-F 2 "" V 7755 3425 50  0001 C CNN
+F 2 "Resistor_SMD:R_0603_1608Metric_Pad0.98x0.95mm_HandSolder" V 7755 3425 50  0001 C CNN
 F 3 "~" H 7825 3425 50  0001 C CNN
 	1    7825 3425
@@
 	3825 3225 4050 3225
 $Comp
-L Device:Resonator Y?
+L Device:Resonator Y1
 U 1 1 5FFC8CC8
 P 3675 4400
-F 0 "Y?" H 3675 4648 50  0000 C CNN
+F 0 "Y1" H 3675 4648 50  0000 C CNN
 F 1 "16MHz" H 3675 4557 50  0000 C CNN
-F 2 "" H 3650 4400 50  0001 C CNN
+F 2 "AERO_CUSTOM:Resonator_SMD_muRata_CSTxExxV-3Pin_3.0x1.1mm_HandSoldering" H 3650 4400 50  0001 C CNN
 F 3 "~" H 3650 4400 50  0001 C CNN
 	1    3675 4400
