File: PacMan/KiCad/Pacman2020/_autosave-precharge.sch (KiCad schematic (older format))
At the start: 15 parts, among them J1 DF22-1P-7.92DSA(05), J2 DF22-1P-7.92DSA(05), J3 DF22-1P-7.92DSA(05), J4 JST PH, K1 G2RL, K2 G5V-1, Q1 MMBT2222A

Commit message: update file names
Parts:
- added R9: R, Resistor_THT:R_Axial_Power_L25.0mm_W9.0mm_P30.48mm, symbol Device:R
- D7: renamed from D3; footprint Package_TO_SOT_SMD:SOT-23_Handsoldering -> Package_TO_SOT_SMD:SOT-23
- Q1: footprint Package_TO_SOT_SMD:SOT-23 -> Package_TO_SOT_SMD:SOT-23_Handsoldering
- R1: footprint Resistor_SMD:R_0603_1608Metric_Pad0.98x0.95mm_HandSolder -> Resistor_THT:R_Axial_Power_L25.0mm_W9.0mm_P30.48mm
Connections:
- net AIR_B+: now also J4.1 (Pin_1); no longer J4.2 (Pin_2)
- net SHDN_IN: now also J4.2 (Pin_2); no longer J4.1 (Pin_1)
- net BAT+: now reaches F2.2, J2.1 (Pin_1)
- net at K1.5, K1.6, R1.1: now also R9.1
- net INT+: now reaches J3.1 (Pin_1), R1.2
- net INT+: now also R9.2
- net INT-: now reaches F1.2, J1.1 (Pin_1)
Changed lines of the file:
@@
 F 0 "R1" V 3293 3450 50  0000 C CNN
 F 1 "R" V 3384 3450 50  0000 C CNN
-F 2 "Resistor_SMD:R_0603_1608Metric_Pad0.98x0.95mm_HandSolder" V 3430 3450 50  0001 C CNN
+F 2 "Resistor_THT:R_Axial_Power_L25.0mm_W9.0mm_P30.48mm" V 3430 3450 50  0001 C CNN
 F 3 "~" H 3500 3450 50  0001 C CNN
 	1    3500 3450
@@
 	3300 2350 2500 2350
 Wire Wire Line
-	3350 3450 2500 3450
+	3350 3450 3125 3450
 $Comp
 L Device:D D1
@@
 F 0 "Q1" H 4616 3696 50  0000 L CNN
 F 1 "MMBT2222A" H 4616 3605 50  0000 L CNN
-F 2 "Package_TO_SOT_SMD:SOT-23" H 4625 3750 50  0001 C CNN
+F 2 "Package_TO_SOT_SMD:SOT-23_Handsoldering" H 4625 3750 50  0001 C CNN
 F 3 "~" H 4425 3650 50  0001 C CNN
 	1    4425 3650
@@
 	1    0    0    -1
 $EndComp
+Text Label 7800 2775 0    50   ~ 0
+AIR_B-
 Text Label 7800 2675 0    50   ~ 0
-AIR_B-
-Text Label 7800 2775 0    50   ~ 0
 AIR_B+
-Text HLabel 7575 2675 0    50   Input ~ 0
+Text HLabel 7575 2775 0    50   Input ~ 0
 SHDN_IN
-Wire Wire Line
-	7575 2675 8150 2675
-Wire Wire Line
-	7800 2775 8350 2775
 Wire Wire Line
 	8625 2875 8550 2875
@@
 	8250 3475 8250 3350
 Wire Wire Line
-	8150 2950 8150 2675
-Connection ~ 8150 2675
-Wire Wire Line
-	8150 2675 8625 2675
-Wire Wire Line
-	8350 2950 8350 2775
-Connection ~ 8350 2775
-Wire Wire Line
-	8350 2775 8625 2775
-Wire Wire Line
 	5050 5150 5050 5500
 $Comp
-L Diode:MMBZxx D3
+L Diode:MMBZxx D7
 U 1 1 601F4E4A
 P 8250 3150
-F 0 "D3" H 7950 3225 50  0000 L CNN
-F 1 "MMBZxx" H 7775 3100 50  0000 L CNN
-F 2 "Package_TO_SOT_SMD:SOT-23_Handsoldering" H 8400 3050 50  0001 L CNN
+F 0 "D7" H 8438 3196 50  0000 L CNN
+F 1 "MMBZxx" H 8438 3105 50  0000 L CNN
+F 2 "Package_TO_SOT_SMD:SOT-23" H 8400 3050 50  0001 L CNN
 F 3 "http://www.onsemi.com/pub/Collateral/MMBZ5V6ALT1-D.PDF" V 8150 3150 50  0001 C CNN
 	1    8250 3150
 	1    0    0    -1
 $EndComp
+$Comp
+L Device:R R?
+U 1 1 60109A97
+P 3500 3650
+AR Path="/60109A97" Ref="R?"  Part="1"
+AR Path="/5FA4E758/60109A97" Ref="R9"  Part="1"
+F 0 "R9" V 3425 3650 50  0000 C CNN
+F 1 "R" V 3625 3625 50  0000 C CNN
+F 2 "Resistor_THT:R_Axial_Power_L25.0mm_W9.0mm_P30.48mm" V 3430 3650 50  0001 C CNN
+F 3 "~" H 3500 3650 50  0001 C CNN
+	1    3500 3650
+	0    1    1    0
+$EndComp
+Wire Wire Line
+	3925 3450 3925 3650
+Wire Wire Line
+	3925 3650 3650 3650
+Connection ~ 3925 3450
+Wire Wire Line
+	3125 3450 3125 3650
+Wire Wire Line
+	3125 3650 3350 3650
+Connection ~ 3125 3450
+Wire Wire Line
+	3125 3450 2500 3450
+Wire Wire Line
+	7800 2675 8350 2675
+Wire Wire Line
+	8150 2950 8150 2775
+Wire Wire Line
+	7575 2775 8150 2775
+Connection ~ 8150 2775
+Wire Wire Line
+	8150 2775 8625 2775
+Wire Wire Line
+	8350 2950 8350 2675
+Connection ~ 8350 2675
+Wire Wire Line
+	8350 2675 8625 2675
+Text Label 2800 1975 0    50   ~ 0
+INT-
+Text Label 2775 2350 0    50   ~ 0
+BAT+
+Text Label 2675 3450 0    50   ~ 0
+INT+
 $EndSCHEMATC
