File: PacMan/KiCad/Pacman2020/precharge.sch (KiCad schematic (older format))
At the start: 17 parts, among them J1 DF22-1P-7.92DSA(05), J2 DF22-1P-7.92DSA(05), J3 DF22-1P-7.92DSA(05), J4 JST PH, K1 G2RL, K2 G5V-1, Q1 MMBT2222A

Commit message: update file names
Parts:
- removed D3, D4: D_Zener, Diode_SMD:D_SMB_Handsoldering, symbol Device:D_Zener
- added R9: R, Resistor_THT:R_Axial_Power_L25.0mm_W9.0mm_P30.48mm, symbol Device:R
- Q1: footprint DigiKey_Lib:SOT-23-3 -> Package_TO_SOT_SMD:SOT-23_Handsoldering
- R1: footprint Resistor_SMD:R_0603_1608Metric_Pad1.05x0.95mm_HandSolder -> Resistor_THT:R_Axial_Power_L25.0mm_W9.0mm_P30.48mm
- R2, R3: footprint Resistor_SMD:R_0603_1608Metric_Pad1.05x0.95mm_HandSolder -> Resistor_SMD:R_0603_1608Metric_Pad0.98x0.95mm_HandSolder
- gave numbers to parts that had none: 1
Connections:
- wire segments 45 -> 48
Other:
- moved on the sheet: D7
Changed lines of the file:
@@
 F 0 "R1" V 3293 3450 50  0000 C CNN
 F 1 "R" V 3384 3450 50  0000 C CNN
-F 2 "Resistor_SMD:R_0603_1608Metric_Pad1.05x0.95mm_HandSolder" V 3430 3450 50  0001 C CNN
+F 2 "Resistor_THT:R_Axial_Power_L25.0mm_W9.0mm_P30.48mm" V 3430 3450 50  0001 C CNN
 F 3 "~" H 3500 3450 50  0001 C CNN
 	1    3500 3450
@@
 	3300 2350 2500 2350
 Wire Wire Line
-	3350 3450 2500 3450
+	3350 3450 3125 3450
 $Comp
 L Device:D D1
@@
 F 0 "Q1" H 4616 3696 50  0000 L CNN
 F 1 "MMBT2222A" H 4616 3605 50  0000 L CNN
-F 2 "DigiKey_Lib:SOT-23-3" H 4625 3750 50  0001 C CNN
+F 2 "Package_TO_SOT_SMD:SOT-23_Handsoldering" H 4625 3750 50  0001 C CNN
 F 3 "~" H 4425 3650 50  0001 C CNN
 	1    4425 3650
@@
 F 0 "R2" V 4568 3650 50  0000 C CNN
 F 1 "R" V 4659 3650 50  0000 C CNN
-F 2 "Resistor_SMD:R_0603_1608Metric_Pad1.05x0.95mm_HandSolder" V 4705 3650 50  0001 C CNN
+F 2 "Resistor_SMD:R_0603_1608Metric_Pad0.98x0.95mm_HandSolder" V 4705 3650 50  0001 C CNN
 F 3 "~" H 4775 3650 50  0001 C CNN
 	1    4775 3650
@@
 F 0 "R3" H 4995 4046 50  0000 L CNN
 F 1 "R" H 4995 3955 50  0000 L CNN
-F 2 "Resistor_SMD:R_0603_1608Metric_Pad1.05x0.95mm_HandSolder" V 4855 4000 50  0001 C CNN
+F 2 "Resistor_SMD:R_0603_1608Metric_Pad0.98x0.95mm_HandSolder" V 4855 4000 50  0001 C CNN
 F 3 "~" H 4925 4000 50  0001 C CNN
 	1    4925 4000
@@
 	1    0    0    -1
 $EndComp
+Text Label 7800 2775 0    50   ~ 0
+AIR_B-
 Text Label 7800 2675 0    50   ~ 0
-AIR_B-
-Text Label 7800 2775 0    50   ~ 0
 AIR_B+
-Text HLabel 7575 2675 0    50   Input ~ 0
+Text HLabel 7575 2775 0    50   Input ~ 0
 SHDN_IN
 Wire Wire Line
-	7575 2675 8150 2675
-Wire Wire Line
-	7800 2775 8325 2775
-$Comp
-L Device:D_Zener D3
-U 1 1 5FAA05CE
-P 8150 3100
-F 0 "D3" V 8075 2850 50  0000 L CNN
-F 1 "D_Zener" V 8200 2700 50  0000 L CNN
-F 2 "Diode_SMD:D_SMB_Handsoldering" H 8150 3100 50  0001 C CNN
-F 3 "~" H 8150 3100 50  0001 C CNN
-	1    8150 3100
-	0    1    1    0
-$EndComp
-$Comp
-L Device:D_Zener D4
-U 1 1 5FAA0C74
-P 8325 3100
-F 0 "D4" V 8225 3175 50  0000 L CNN
-F 1 "D_Zener" V 8375 2700 50  0001 L CNN
-F 2 "Diode_SMD:D_SMB_Handsoldering" H 8325 3100 50  0001 C CNN
-F 3 "~" H 8325 3100 50  0001 C CNN
-	1    8325 3100
-	0    1    1    0
-$EndComp
+	7800 2675 8150 2675
+Wire Wire Line
+	7575 2775 8350 2775
 Wire Wire Line
 	8625 2875 8550 2875
@@
 L power:GND #PWR0102
 U 1 1 5FAA23F0
-P 8250 3375
-F 0 "#PWR0102" H 8250 3125 50  0001 C CNN
-F 1 "GND" H 8255 3202 50  0000 C CNN
-F 2 "" H 8250 3375 50  0001 C CNN
-F 3 "" H 8250 3375 50  0001 C CNN
-	1    8250 3375
+P 8250 3475
+F 0 "#PWR0102" H 8250 3225 50  0001 C CNN
+F 1 "GND" H 8255 3302 50  0000 C CNN
+F 2 "" H 8250 3475 50  0001 C CNN
+F 3 "" H 8250 3475 50  0001 C CNN
+	1    8250 3475
 	1    0    0    -1
 $EndComp
@@
 Connection ~ 8550 2975
 Wire Wire Line
-	8250 3375 8250 3250
-Wire Wire Line
-	8250 3250 8325 3250
-Wire Wire Line
-	8250 3250 8150 3250
-Connection ~ 8250 3250
+	8250 3475 8250 3350
 Wire Wire Line
 	8150 2950 8150 2675
@@
 	8150 2675 8625 2675
 Wire Wire Line
-	8325 2950 8325 2775
-Connection ~ 8325 2775
-Wire Wire Line
-	8325 2775 8625 2775
+	8350 2950 8350 2775
+Connection ~ 8350 2775
+Wire Wire Line
+	8350 2775 8625 2775
 Wire Wire Line
 	5050 5150 5050 5500
 $Comp
-L Diode:MMBZxx D?
+L Diode:MMBZxx D7
 U 1 1 601F4E4A
-P 7425 3425
-F 0 "D?" H 7613 3471 50  0000 L CNN
-F 1 "MMBZxx" H 7613 3380 50  0000 L CNN
-F 2 "Package_TO_SOT_SMD:SOT-23" H 7575 3325 50  0001 L CNN
-F 3 "http://www.onsemi.com/pub/Collateral/MMBZ5V6ALT1-D.PDF" V 7325 3425 50  0001 C CNN
-	1    7425 3425
-	1    0    0    -1
-$EndComp
+P 8250 3150
+F 0 "D7" H 8438 3196 50  0000 L CNN
+F 1 "MMBZxx" H 8438 3105 50  0000 L CNN
+F 2 "Package_TO_SOT_SMD:SOT-23" H 8400 3050 50  0001 L CNN
+F 3 "http://www.onsemi.com/pub/Collateral/MMBZ5V6ALT1-D.PDF" V 8150 3150 50  0001 C CNN
+	1    8250 3150
+	1    0    0    -1
+$EndComp
+$Comp
+L Device:R R?
+U 1 1 60109A97
+P 3500 3650
+AR Path="/60109A97" Ref="R?"  Part="1"
+AR Path="/5FA4E758/60109A97" Ref="R9"  Part="1"
+F 0 "R9" V 3425 3650 50  0000 C CNN
+F 1 "R" V 3625 3625 50  0000 C CNN
+F 2 "Resistor_THT:R_Axial_Power_L25.0mm_W9.0mm_P30.48mm" V 3430 3650 50  0001 C CNN
+F 3 "~" H 3500 3650 50  0001 C CNN
+	1    3500 3650
+	0    1    1    0
+$EndComp
+Wire Wire Line
+	3925 3450 3925 3650
+Wire Wire Line
+	3925 3650 3650 3650
+Connection ~ 3925 3450
+Wire Wire Line
+	3125 3450 3125 3650
+Wire Wire Line
+	3125 3650 3350 3650
+Connection ~ 3125 3450
+Wire Wire Line
+	3125 3450 2500 3450
 $EndSCHEMATC

Commit message: layout changes
Connections:
- net GND: now also Q1.2 (E), R3.2
- net BATT+: now reaches F2.2, J2.1 (Pin_1)
- net INT+: now reaches J3.1 (Pin_1), R1.2, R9.2
- net INT-: now reaches F1.2, J1.1 (Pin_1)
Other:
- note added: "1k 7W\nin parallel"
- note added: "AIR+ Relay signal"
- note added: "BATT+"
- note added: "Connector for AIR+/- signal"
- note added: "INT+"
- note added: "INT-"
- note added: "Precharge Order\n- Shutdown loop in, closes AIR -\n- Precharge relay (from Rinehart signal), Connects BATT+ to INT+\n- Main Contactor (from Rinehart signal), clses AIR+\n\nINT+/- are connected to the RineHart +/- Inputs"
- note added: "Precharge relay"
- moved on the sheet: D1, D2, D7, F1, F2, J1, J2, J3, J4, K1, K2, Q1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
