File: LVPDU/KiCad/LVPDU.sch (KiCad schematic (older format))
At the start: 12 parts, among them K1 T9VV1K15-12S

Commit message: inital layouts
Parts:
- D1: footprint (none) -> Package_TO_SOT_THT:TO-220-3_Horizontal_TabUp
- F1, F2, F3, F4, F5, F6, F7: footprint (none) -> AERO_CUSTOM:Fuseholder_Blade_Mini_Keystone_3568
- H1, H2: renamed from H?; footprint (none) -> MountingHole:MountingHole_3.2mm_M3
- J1: renamed from J?; footprint (none) -> AERO_CUSTOM:TE_1-776266-1_14pin_Horizontal
- K1: footprint AERO-footprints:RELAY_T9VV1K15-12S -> AERO_CUSTOM:RELAY_T9VV1K15-12S
Changed lines of the file:
@@
 F 0 "F1" V 9678 1375 50  0000 C CNN
 F 1 "3568 Mini Blade" V 9769 1375 50  0000 C CNN
-F 2 "" V 9805 1375 50  0001 C CNN
+F 2 "AERO_CUSTOM:Fuseholder_Blade_Mini_Keystone_3568" V 9805 1375 50  0001 C CNN
 F 3 "~" H 9875 1375 50  0001 C CNN
 	1    9875 1375
@@
 F 0 "F2" V 9678 1675 50  0000 C CNN
 F 1 "3568 Mini Blade" V 9769 1675 50  0000 C CNN
-F 2 "" V 9805 1675 50  0001 C CNN
+F 2 "AERO_CUSTOM:Fuseholder_Blade_Mini_Keystone_3568" V 9805 1675 50  0001 C CNN
 F 3 "~" H 9875 1675 50  0001 C CNN
 	1    9875 1675
@@
 F 0 "F3" V 9678 1975 50  0000 C CNN
 F 1 "3568 Mini Blade" V 9769 1975 50  0000 C CNN
-F 2 "" V 9805 1975 50  0001 C CNN
+F 2 "AERO_CUSTOM:Fuseholder_Blade_Mini_Keystone_3568" V 9805 1975 50  0001 C CNN
 F 3 "~" H 9875 1975 50  0001 C CNN
 	1    9875 1975
@@
 F 0 "F4" V 9678 2275 50  0000 C CNN
 F 1 "3568 Mini Blade" V 9769 2275 50  0000 C CNN
-F 2 "" V 9805 2275 50  0001 C CNN
+F 2 "AERO_CUSTOM:Fuseholder_Blade_Mini_Keystone_3568" V 9805 2275 50  0001 C CNN
 F 3 "~" H 9875 2275 50  0001 C CNN
 	1    9875 2275
@@
 F 0 "F5" V 9678 2600 50  0000 C CNN
 F 1 "3568 Mini Blade" V 9769 2600 50  0000 C CNN
-F 2 "" V 9805 2600 50  0001 C CNN
+F 2 "AERO_CUSTOM:Fuseholder_Blade_Mini_Keystone_3568" V 9805 2600 50  0001 C CNN
 F 3 "~" H 9875 2600 50  0001 C CNN
 	1    9875 2600
@@
 F 0 "F6" V 9678 2950 50  0000 C CNN
 F 1 "3568 Mini Blade" V 9769 2950 50  0000 C CNN
-F 2 "" V 9805 2950 50  0001 C CNN
+F 2 "AERO_CUSTOM:Fuseholder_Blade_Mini_Keystone_3568" V 9805 2950 50  0001 C CNN
 F 3 "~" H 9875 2950 50  0001 C CNN
 	1    9875 2950
@@
 F 0 "K1" V 6767 4375 50  0000 C CNN
 F 1 "T9VV1K15-12S" V 6676 4375 50  0000 C CNN
-F 2 "AERO-footprints:RELAY_T9VV1K15-12S" H 6650 4325 50  0001 L CNN
+F 2 "AERO_CUSTOM:RELAY_T9VV1K15-12S" H 6650 4325 50  0001 L CNN
 F 3 "https://www.te.com/commerce/DocumentDelivery/DDEController?Action=srchrtrv&DocNm=Power_PCB_Relay_T9V_Solar&DocType=DS&DocLang=English" H 6300 4375 50  0001 C CNN
 	1    6300 4375
@@
 F 0 "F7" V 9678 3525 50  0000 C CNN
 F 1 "3568 Mini Blade" V 9769 3525 50  0000 C CNN
-F 2 "" V 9805 3525 50  0001 C CNN
+F 2 "AERO_CUSTOM:Fuseholder_Blade_Mini_Keystone_3568" V 9805 3525 50  0001 C CNN
 F 3 "~" H 9875 3525 50  0001 C CNN
 	1    9875 3525
@@
 F 0 "D1" H 6300 5881 50  0000 C CNN
 F 1 "D_Schottky_AKA" H 6300 5790 50  0000 C CNN
-F 2 "" H 6275 5600 50  0001 C CNN
+F 2 "Package_TO_SOT_THT:TO-220-3_Horizontal_TabUp" H 6275 5600 50  0001 C CNN
 F 3 "~" H 6275 5600 50  0001 C CNN
 	1    6275 5600
@@
 BATT_IN
 $Comp
-L power:GND #PWR?
+L power:GND #PWR0104
 U 1 1 5FFE7EE3
 P 9550 5525
-F 0 "#PWR?" H 9550 5275 50  0001 C CNN
+F 0 "#PWR0104" H 9550 5275 50  0001 C CNN
 F 1 "GND" H 9555 5352 50  0000 C CNN
 F 2 "" H 9550 5525 50  0001 C CNN
@@
 $EndComp
 $Comp
-L Connector_Generic:Conn_01x14 J?
+L Connector_Generic:Conn_01x14 J1
 U 1 1 5FFF0982
 P 10400 4825
-F 0 "J?" H 10480 4817 50  0000 L CNN
+F 0 "J1" H 10480 4817 50  0000 L CNN
 F 1 "Conn_01x14" H 10480 4726 50  0000 L CNN
-F 2 "" H 10400 4825 50  0001 C CNN
+F 2 "AERO_CUSTOM:TE_1-776266-1_14pin_Horizontal" H 10400 4825 50  0001 C CNN
 F 3 "~" H 10400 4825 50  0001 C CNN
 	1    10400 4825
@@
 	5175 4175 6000 4175
 $Comp
-L Mechanical:MountingHole H?
+L Mechanical:MountingHole H1
 U 1 1 6000AF10
 P 5925 6975
-F 0 "H?" H 6025 7021 50  0000 L CNN
+F 0 "H1" H 6025 7021 50  0000 L CNN
 F 1 "MountingHole" H 6025 6930 50  0000 L CNN
-F 2 "" H 5925 6975 50  0001 C CNN
+F 2 "MountingHole:MountingHole_3.2mm_M3" H 5925 6975 50  0001 C CNN
 F 3 "~" H 5925 6975 50  0001 C CNN
 	1    5925 6975
@@
 $EndComp
 $Comp
-L Mechanical:MountingHole H?
+L Mechanical:MountingHole H2
 U 1 1 6000C4CB
 P 5925 7375
-F 0 "H?" H 6025 7421 50  0000 L CNN
+F 0 "H2" H 6025 7421 50  0000 L CNN
 F 1 "MountingHole" H 6025 7330 50  0000 L CNN
-F 2 "" H 5925 7375 50  0001 C CNN
+F 2 "MountingHole:MountingHole_3.2mm_M3" H 5925 7375 50  0001 C CNN
 F 3 "~" H 5925 7375 50  0001 C CNN
 	1    5925 7375

Commit message: first board rev
Parts:
- added F8, F9: 3568 Mini Blade, AERO_CUSTOM:Fuseholder_Blade_Mini_Keystone_3568, symbol Device:Fuse
- J1: footprint AERO_CUSTOM:TE_1-776266-1_14pin_Horizontal -> AERO_CUSTOM:TE_1-776262-1_14pin_Vertical
Connections:
- net +12V: now also F7.1
- net BATT_IN: now also J1.6 (Pin_6), F8.2; no longer F7.2, J1.11 (Pin_11)
- net DCDC_IN: now also J1.7 (Pin_7), F9.1; no longer D1.1 (A), D1.3 (A), J1.13 (Pin_13)
- net FROM_BRB: now also J1.13 (Pin_13); no longer J1.9 (Pin_9)
- net GND: now also J1.8 (Pin_8); no longer J1.14 (Pin_14)
- net PUMP: now also J1.1 (Pin_1); no longer J1.5 (Pin_5)
- net RADIATOR: now also J1.3 (Pin_3); no longer J1.4 (Pin_4)
- net RINEHART: now also J1.5 (Pin_5); no longer J1.3 (Pin_3)
- net SHUTDOWN_OUT: now also J1.9 (Pin_9); no longer J1.1 (Pin_1)
- net TO_BRB: now also J1.11 (Pin_11), F8.1; no longer F7.1, J1.8 (Pin_8)
- removed net 12V_OUT: F6.2, J1.6 (Pin_6), J1.7 (Pin_7)
- new net 12V_OUT_1: F6.2, J1.4 (Pin_4)
- new net 12V_OUT_2: F7.2, J1.14 (Pin_14)
- new net DCDC_Fused: D1.1 (A), D1.3 (A), F9.2
Other:
- note added: "BATT_IN comes directly from the BRB\nShutdown out goes to the rest of the safety loop\nDCDC_IN comes from DCDC through a fuse. Runs in || with BATT_IN\nDAQ out is the LV Boards\nBoth 12V out are extra 12V outputs"
Changed lines of the file:
@@
 PUMP
 Text Label 9050 2950 0    50   ~ 0
-12V_OUT
+12V_OUT_1
 Wire Wire Line
 	9050 2950 9725 2950
@@
 	0    1    -1   0
 $EndComp
-$Comp
-L Device:Fuse F7
-U 1 1 5FFBD610
-P 9875 3525
-F 0 "F7" V 9678 3525 50  0000 C CNN
-F 1 "3568 Mini Blade" V 9769 3525 50  0000 C CNN
-F 2 "AERO_CUSTOM:Fuseholder_Blade_Mini_Keystone_3568" V 9805 3525 50  0001 C CNN
-F 3 "~" H 9875 3525 50  0001 C CNN
-	1    9875 3525
-	0    1    1    0
-$EndComp
-Text Label 9350 3525 0    50   ~ 0
-BATT_IN
-Wire Wire Line
-	9350 3525 9725 3525
-Text Label 10350 3525 2    50   ~ 0
-TO_BRB
-Wire Wire Line
-	10350 3525 10025 3525
 Text Label 7050 4575 2    50   ~ 0
 FROM_BRB
@@
 	1    0    0    -1
 $EndComp
-Text Label 9550 4225 0    50   ~ 0
+Text Label 9550 5025 0    50   ~ 0
 SHUTDOWN_OUT
 Text Label 9550 4325 0    50   ~ 0
 DAQ
+Text Label 9550 4625 0    50   ~ 0
+RINEHART
 Text Label 9550 4425 0    50   ~ 0
-RINEHART
+RADIATOR
+Text Label 9550 4225 0    50   ~ 0
+PUMP
 Text Label 9550 4525 0    50   ~ 0
-RADIATOR
-Text Label 9550 4625 0    50   ~ 0
-PUMP
+12V_OUT_1
 Text Label 9550 4725 0    50   ~ 0
-12V_OUT
-Text Label 9550 4925 0    50   ~ 0
-TO_BRB
-Text Label 9550 5125 0    50   ~ 0
-BATT_IN
-Text Label 9550 5025 0    50   ~ 0
-FROM_BRB
+BATT_IN
+Text Label 9550 5525 0    50   ~ 0
+12V_OUT_2
 Text Label 9550 5325 0    50   ~ 0
 DCDC_IN
-Text Label 9550 4825 0    50   ~ 0
-12V_OUT
-Text Label 9550 5425 0    50   ~ 0
-DCDC_IN
-Text Label 9550 5225 0    50   ~ 0
+Text Label 9550 5125 0    50   ~ 0
 BATT_IN
 $Comp
 L power:GND #PWR0104
 U 1 1 5FFE7EE3
-P 9550 5525
-F 0 "#PWR0104" H 9550 5275 50  0001 C CNN
-F 1 "GND" H 9555 5352 50  0000 C CNN
-F 2 "" H 9550 5525 50  0001 C CNN
-F 3 "" H 9550 5525 50  0001 C CNN
-	1    9550 5525
+P 9400 4925
+F 0 "#PWR0104" H 9400 4675 50  0001 C CNN
+F 1 "GND" H 9405 4752 50  0000 C CNN
+F 2 "" H 9400 4925 50  0001 C CNN
+F 3 "" H 9400 4925 50  0001 C CNN
+	1    9400 4925
 	1    0    0    -1
 $EndComp
@@
 F 0 "J1" H 10480 4817 50  0000 L CNN
 F 1 "Conn_01x14" H 10480 4726 50  0000 L CNN
-F 2 "AERO_CUSTOM:TE_1-776266-1_14pin_Horizontal" H 10400 4825 50  0001 C CNN
+F 2 "AERO_CUSTOM:TE_1-776262-1_14pin_Vertical" H 10400 4825 50  0001 C CNN
 F 3 "~" H 10400 4825 50  0001 C CNN
 	1    10400 4825
@@
 $EndComp
 Wire Wire Line
+	10200 5025 9550 5025
+Wire Wire Line
+	10200 4325 9550 4325
+Wire Wire Line
+	9550 4625 10200 4625
+Wire Wire Line
+	10200 4425 9550 4425
+Wire Wire Line
 	10200 4225 9550 4225
 Wire Wire Line
-	10200 4325 9550 4325
-Wire Wire Line
-	9550 4425 10200 4425
-Wire Wire Line
 	10200 4525 9550 4525
 Wire Wire Line
-	10200 4625 9550 4625
+	10200 5525 9550 5525
 Wire Wire Line
 	10200 4725 9550 4725
 Wire Wire Line
-	10200 4825 9550 4825
-Wire Wire Line
-	10200 4925 9550 4925
-Wire Wire Line
-	10200 5025 9550 5025
-Wire Wire Line
 	10200 5125 9550 5125
 Wire Wire Line
-	10200 5225 9550 5225
-Wire Wire Line
 	10200 5325 9550 5325
 Wire Wire Line
-	10200 5425 9550 5425
-Wire Wire Line
-	10200 5525 9550 5525
-Text Label 5575 4175 0    50   ~ 0
-MAIN_GLV
-Text Label 6900 5550 2    50   ~ 0
+	10200 4925 9400 4925
+Text Label 8100 5550 2    50   ~ 0
 DCDC_IN
-Wire Wire Line
-	6900 5550 6475 5550
 Wire Wire Line
 	6475 5550 6475 5500
@@
 	6475 5550 6475 5600
 Connection ~ 6475 5550
-Text Label 5650 5600 0    50   ~ 0
-MAIN_GLV
 Wire Wire Line
 	5650 5600 6125 5600
@@
 	1    0    0    -1
 $EndComp
+Text Notes 3875 3025 0    94   ~ 0
+BATT_IN comes directly from the BRB\nShutdown out goes to the rest of the safety loop\nDCDC_IN comes from DCDC through a fuse. Runs in || with BATT_IN\nDAQ out is the LV Boards\nBoth 12V out are extra 12V outputs
+Text Label 9550 5425 0    50   ~ 0
+FROM_BRB
+Text Label 9550 5225 0    50   ~ 0
+TO_BRB
+Wire Wire Line
+	9550 5425 10200 5425
+Wire Wire Line
+	10200 5225 9550 5225
+$Comp
+L Device:Fuse F7
+U 1 1 602183CF
+P 9875 3300
+F 0 "F7" V 9678 3300 50  0000 C CNN
+F 1 "3568 Mini Blade" V 9769 3300 50  0000 C CNN
+F 2 "AERO_CUSTOM:Fuseholder_Blade_Mini_Keystone_3568" V 9805 3300 50  0001 C CNN
+F 3 "~" H 9875 3300 50  0001 C CNN
+	1    9875 3300
+	0    1    1    0
+$EndComp
+Text Label 9050 3300 0    50   ~ 0
+12V_OUT_2
+Wire Wire Line
+	9050 3300 9725 3300
+Wire Wire Line
+	10350 3300 10025 3300
+Connection ~ 10350 2950
+Wire Wire Line
+	10350 3300 10350 2950
+$Comp
+L Device:Fuse F8
+U 1 1 6021FB68
+P 9900 3800
+F 0 "F8" V 9703 3800 50  0000 C CNN
+F 1 "3568 Mini Blade" V 9794 3800 50  0000 C CNN
+F 2 "AERO_CUSTOM:Fuseholder_Blade_Mini_Keystone_3568" V 9830 3800 50  0001 C CNN
+F 3 "~" H 9900 3800 50  0001 C CNN
+	1    9900 3800
+	0    1    1    0
+$EndComp
+Text Label 9075 3800 0    50   ~ 0
+BATT_IN
+Wire Wire Line
+	9075 3800 9750 3800
+Wire Wire Line
+	10425 3800 10050 3800
+Text Label 10425 3800 2    50   ~ 0
+TO_BRB
+Text Label 7050 5550 2    50   ~ 0
+DCDC_Fused
+$Comp
+L Device:Fuse F9
+U 1 1 6023B958
+P 7375 5550
+F 0 "F9" V 7178 5550 50  0000 C CNN
+F 1 "3568 Mini Blade" V 7269 5550 50  0000 C CNN
+F 2 "AERO_CUSTOM:Fuseholder_Blade_Mini_Keystone_3568" V 7305 5550 50  0001 C CNN
+F 3 "~" H 7375 5550 50  0001 C CNN
+	1    7375 5550
+	0    1    1    0
+$EndComp
+Wire Wire Line
+	6475 5550 7225 5550
+Wire Wire Line
+	7525 5550 8100 5550
+Text Label 5650 5600 0    50   ~ 0
+BATT_IN
+Wire Wire Line
+	10200 4825 9550 4825
+Text Label 9550 4825 0    50   ~ 0
+DCDC_IN
 $EndSCHEMATC

Commit message: minor update thing
Parts:
- removed H2: MountingHole, MountingHole:MountingHole_3.2mm_M3, symbol Mechanical:MountingHole
- D1: footprint Package_TO_SOT_THT:TO-220-3_Horizontal_TabUp -> Package_TO_SOT_THT:TO-220-3_Horizontal_TabDown
Changed lines of the file:
@@
 F 0 "D1" H 6300 5881 50  0000 C CNN
 F 1 "D_Schottky_AKA" H 6300 5790 50  0000 C CNN
-F 2 "Package_TO_SOT_THT:TO-220-3_Horizontal_TabUp" H 6275 5600 50  0001 C CNN
+F 2 "Package_TO_SOT_THT:TO-220-3_Horizontal_TabDown" H 6275 5600 50  0001 C CNN
 F 3 "~" H 6275 5600 50  0001 C CNN
 	1    6275 5600
@@
 	1    0    0    -1
 $EndComp
-$Comp
-L Mechanical:MountingHole H2
-U 1 1 6000C4CB
-P 5925 7375
-F 0 "H2" H 6025 7421 50  0000 L CNN
-F 1 "MountingHole" H 6025 7330 50  0000 L CNN
-F 2 "MountingHole:MountingHole_3.2mm_M3" H 5925 7375 50  0001 C CNN
-F 3 "~" H 5925 7375 50  0001 C CNN
-	1    5925 7375
-	1    0    0    -1
-$EndComp
