File: LVPDU/KiCad/LVPDU.sch (KiCad schematic (older format))
At the start: 14 parts, among them J1 Conn_01x14, K1 T9VV1K15-12S

Commit message: add contact note
Parts:
- removed H2: MountingHole, MountingHole:MountingHole_3.2mm_M3, symbol Mechanical:MountingHole
- D1: footprint Package_TO_SOT_THT:TO-220-3_Horizontal_TabUp -> Package_TO_SOT_THT:TO-220-3_Horizontal_TabDown
- K1: symbol AERO_custom_symbols:T9VV1K15-12S -> LVPDU-rescue:T9VV1K15-12S-AERO_custom_symbols
Other:
- note added: "All Ampseal Pins\nNeed to Be Gold Plated\nfor Current Rating"
Changed lines of the file:
@@
 	10350 1375 10350 1675
 $Comp
-L AERO_custom_symbols:T9VV1K15-12S K1
+L LVPDU-rescue:T9VV1K15-12S-AERO_custom_symbols K1
 U 1 1 5FFBBBA5
 P 6300 4375
@@
 F 0 "D1" H 6300 5881 50  0000 C CNN
 F 1 "D_Schottky_AKA" H 6300 5790 50  0000 C CNN
-F 2 "Package_TO_SOT_THT:TO-220-3_Horizontal_TabUp" H 6275 5600 50  0001 C CNN
+F 2 "Package_TO_SOT_THT:TO-220-3_Horizontal_TabDown" H 6275 5600 50  0001 C CNN
 F 3 "~" H 6275 5600 50  0001 C CNN
 	1    6275 5600
@@
 	1    0    0    -1
 $EndComp
-$Comp
-L Mechanical:MountingHole H2
-U 1 1 6000C4CB
-P 5925 7375
-F 0 "H2" H 6025 7421 50  0000 L CNN
-F 1 "MountingHole" H 6025 7330 50  0000 L CNN
-F 2 "MountingHole:MountingHole_3.2mm_M3" H 5925 7375 50  0001 C CNN
-F 3 "~" H 5925 7375 50  0001 C CNN
-	1    5925 7375
-	1    0    0    -1
-$EndComp
 Text Notes 3875 3025 0    94   ~ 0
 BATT_IN comes directly from the BRB\nShutdown out goes to the rest of the safety loop\nDCDC_IN comes from DCDC through a fuse. Runs in || with BATT_IN\nDAQ out is the LV Boards\nBoth 12V out are extra 12V outputs
@@
 Text Label 9550 4825 0    50   ~ 0
 DCDC_IN
+Text Notes 9575 5950 0    50   ~ 0
+All Ampseal Pins\nNeed to Be Gold Plated\nfor Current Rating
 $EndSCHEMATC

Commit message: notes from design review 1
Other:
- note added: "TODO: \nAdd fuse for Battery In"
Changed lines of the file:
@@
 Text Notes 9575 5950 0    50   ~ 0
 All Ampseal Pins\nNeed to Be Gold Plated\nfor Current Rating
+Text Notes 4175 6275 0    50   ~ 0
+TODO: \nAdd fuse for Battery In
 $EndSCHEMATC

Commit message: Add Fuse Ratings
Other:
- note added: "10A"
- note added: "2A"
- note added: "30A"
- note added: "5A"
- note added: "7.5A"
Changed lines of the file:
@@
 Text Notes 4175 6275 0    50   ~ 0
 TODO: \nAdd fuse for Battery In
+Text Notes 9650 2700 0    50   ~ 0
+10A
+Text Notes 9650 1750 0    50   ~ 0
+5A
+Text Notes 9650 3050 0    50   ~ 0
+5A
+Text Notes 9650 3400 0    50   ~ 0
+2A
+Text Notes 7300 5700 0    50   ~ 0
+30A
+Text Notes 9650 1450 0    50   ~ 0
+2A
+Text Notes 9600 2350 0    50   ~ 0
+7.5A
+Text Notes 9650 2050 0    50   ~ 0
+5A
 $EndSCHEMATC
