File: LVPDU/KiCad/_autosave-LVPDU.kicad_pcb (KiCad board)
At the start: 2 copper layers, 97.8 x 52.1 mm, 13 parts, among them J1 Conn_01x14, K1 T9VV1K15-12S

Commit message: gerber files
Parts:
- added G***: LOGO, AERO_CUSTOM:AERO_Logo_10x4mm, F.Cu at (237.5, 74.3)
Changed lines of the file:
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@@
     (tracks 183)
     (zones 0)
-    (modules 13)
+    (modules 14)
     (nets 15)
   )
@@
   )
   (setup
-    (last_trace_width 2.4)
+    (last_trace_width 0.25)
     (user_trace_width 0.8)
     (user_trace_width 1)
@@
       (outputformat 1)
       (mirror false)
-      (drillshape 1)
+      (drillshape 0)
       (scaleselection 1)
-      (outputdirectory ""))
+      (outputdirectory "LVPDU_Gerber/"))
   )
   (net 0 "")
@@
     (add_net GND)
   )
+  (module AERO_CUSTOM:AERO_Logo_10x4mm (layer F.Cu)
+    (at 237.49 74.295 90)
+    (fp_text reference G*** (at 0 0 90) (layer F.SilkS) hide
+      (effects (font (size 1.524 1.524) (thickness 0.3)))
+    )
+    (fp_text value LOGO (at 0.75 0 90) (layer F.SilkS) hide
+      (effects (font (size 1.524 1.524) (thickness 0.3)))
+    )
+    (fp_poly (pts (xy 4.590646 -1.503024) (xy 5.010092 -1.084064) (xy 5.010092 1.01413) (xy 4.135758 1.887556)
+      (xy 3.745677 1.496968) (xy 3.355597 1.106381) (xy 3.355597 0.91824) (xy 3.938166 0.91824)
+      (xy 4.012973 0.995422) (xy 4.087781 1.072604) (xy 4.246001 0.915597) (xy 4.404221 0.758589)
+      (xy 4.404221 -0.804819) (xy 4.171193 -1.036973) (xy 3.938166 -1.269126) (xy 3.938166 0.91824)
+      (xy 3.355597 0.91824) (xy 3.355597 -1.10738) (xy 3.763398 -1.514682) (xy 4.1712 -1.921985)
+      (xy 4.590646 -1.503024)) (layer F.SilkS) (width 0.01))
+    (fp_poly (pts (xy 3.052661 -1.246114) (xy 3.052661 -0.641748) (xy 2.645809 -0.233002) (xy 2.860886 -0.017026)
+      (xy 3.075964 0.198949) (xy 3.075964 1.105415) (xy 3.197841 1.228826) (xy 3.319719 1.352236)
+      (xy 3.051947 1.620008) (xy 2.784175 1.887779) (xy 2.261465 1.363211) (xy 2.491377 1.106881)
+      (xy 2.492386 0.803547) (xy 2.493395 0.500214) (xy 2.237065 0.244679) (xy 1.980734 -0.010857)
+      (xy 1.980734 1.131935) (xy 2.097505 1.246951) (xy 2.214276 1.361966) (xy 1.952243 1.624744)
+      (xy 1.862409 1.713933) (xy 1.783925 1.790151) (xy 1.722682 1.847811) (xy 1.684576 1.881323)
+      (xy 1.675144 1.887523) (xy 1.654733 1.87152) (xy 1.608141 1.827324) (xy 1.541156 1.760657)
+      (xy 1.459566 1.677241) (xy 1.405051 1.620528) (xy 1.150023 1.353533) (xy 1.274094 1.231003)
+      (xy 1.398166 1.108473) (xy 1.398166 -0.314816) (xy 1.934129 -0.314816) (xy 2.231125 -0.611812)
+      (xy 2.528121 -0.908807) (xy 1.934129 -1.502799) (xy 1.934129 -0.314816) (xy 1.398166 -0.314816)
+      (xy 1.398166 -1.175438) (xy 1.264759 -1.310251) (xy 1.131352 -1.445065) (xy 1.363358 -1.677945)
+      (xy 1.595365 -1.910826) (xy 2.389135 -1.910826) (xy 3.052661 -1.246114)) (layer F.SilkS) (width 0.01))
+    (fp_poly (pts (xy -1.416608 -1.47486) (xy -0.991063 -1.048849) (xy -1.21171 -0.827281) (xy -1.432356 -0.605713)
+      (xy -2.073944 -1.246073) (xy -2.073944 -0.277684) (xy -1.189008 -0.291284) (xy -1.473833 -0.005826)
+      (xy -1.758658 0.279633) (xy -2.073944 0.279633) (xy -2.073944 0.953041) (xy -1.990882 1.016396)
+      (xy -1.90782 1.07975) (xy -1.432564 0.606112) (xy -1.01212 1.026556) (xy -1.444776 1.457039)
+      (xy -1.561006 1.57228) (xy -1.666275 1.675877) (xy -1.75613 1.763512) (xy -1.82612 1.830866)
+      (xy -1.871792 1.873621) (xy -1.888568 1.887523) (xy -1.907491 1.871751) (xy -1.954481 1.827522)
+      (xy -2.024781 1.759462) (xy -2.113633 1.672199) (xy -2.21628 1.570361) (xy -2.278108 1.508596)
+      (xy -2.656513 1.129669) (xy -2.656513 -1.081938) (xy -2.249333 -1.491404) (xy -1.842152 -1.900871)
+      (xy -1.416608 -1.47486)) (layer F.SilkS) (width 0.01))
+    (fp_poly (pts (xy -3.477698 -1.508623) (xy -3.075963 -1.106395) (xy -3.075963 1.105415) (xy -2.954085 1.228826)
+      (xy -2.832208 1.352236) (xy -3.09998 1.620008) (xy -3.367752 1.887779) (xy -3.902032 1.351979)
+      (xy -3.658532 1.105415) (xy -3.658532 0.629174) (xy -4.171192 0.629174) (xy -4.171192 1.105415)
+      (xy -4.049315 1.228826) (xy -3.927437 1.352236) (xy -4.195209 1.620008) (xy -4.462981 1.887779)
+      (xy -4.997261 1.351979) (xy -4.753761 1.105415) (xy -4.753761 0.023303) (xy -4.171192 0.023303)
+      (xy -3.658532 0.023303) (xy -3.658532 -0.735332) (xy -3.913681 -1.002666) (xy -4.168831 -1.27)
+      (xy -4.170011 -0.623349) (xy -4.171192 0.023303) (xy -4.753761 0.023303) (xy -4.753761 -1.037433)
+      (xy -4.316597 -1.474142) (xy -3.879434 -1.910851) (xy -3.477698 -1.508623)) (layer F.SilkS) (width 0.01))
+    (fp_poly (pts (xy 0.594221 -1.374862) (xy 0.354968 -0.722385) (xy 0.717059 -0.722385) (xy 0.853644 -0.722106)
+      (xy 0.949683 -0.720764) (xy 1.011233 -0.717601) (xy 1.044352 -0.711857) (xy 1.055098 -0.702775)
+      (xy 1.049529 -0.689597) (xy 1.04285 -0.681606) (xy 1.024199 -0.657081) (xy 0.981096 -0.598426)
+      (xy 0.91624 -0.509389) (xy 0.83233 -0.39372) (xy 0.732061 -0.25517) (xy 0.618134 -0.097489)
+      (xy 0.493246 0.075575) (xy 0.360094 0.26027) (xy 0.221378 0.452846) (xy 0.079794 0.649555)
+      (xy -0.061959 0.846645) (xy -0.201183 1.040368) (xy -0.33518 1.226972) (xy -0.461252 1.402708)
+      (xy -0.576701 1.563827) (xy -0.67883 1.706578) (xy -0.764939 1.827211) (xy -0.832331 1.921976)
+      (xy -0.878309 1.987123) (xy -0.900173 2.018903) (xy -0.900652 2.019655) (xy -0.898812 2.007273)
+      (xy -0.882983 1.955011) (xy -0.854541 1.86699) (xy -0.814862 1.74733) (xy -0.765324 1.600151)
+      (xy -0.707302 1.429575) (xy -0.642173 1.23972) (xy -0.580239 1.060454) (xy -0.509049 0.854915)
+      (xy -0.442772 0.663314) (xy -0.382925 0.490054) (xy -0.331024 0.33954) (xy -0.288589 0.216175)
+      (xy -0.257135 0.124363) (xy -0.23818 0.068509) (xy -0.233027 0.05261) (xy -0.254981 0.050511)
+      (xy -0.315447 0.048732) (xy -0.406333 0.047414) (xy -0.519545 0.046696) (xy -0.579325 0.046605)
+      (xy -0.925622 0.046605) (xy -0.665354 -0.541789) (xy -0.583068 -0.727996) (xy -0.494257 -0.929277)
+      (xy -0.404488 -1.132995) (xy -0.319327 -1.326516) (xy -0.244339 -1.497202) (xy -0.208576 -1.578762)
+      (xy -0.012066 -2.027339) (xy 0.833473 -2.027339) (xy 0.594221 -1.374862)) (layer F.SilkS) (width 0.01))
+  )
   (module Package_TO_SOT_THT:TO-220-3_Horizontal_TabDown (layer F.Cu)
     (at 147.828 60.856)
@@
     )
     (fp_text value D_Schottky_AKA (at 2.54 2) (layer F.Fab)
-      (effects (font (size 1 1) (thickness 0.15)))
-    )
-    (fp_text user %R (at 2.54 -20.58) (layer F.Fab)
       (effects (font (size 1 1) (thickness 0.15)))
     )
@@
     (fp_line (start 7.79 1.25) (end 7.79 -19.71) (layer F.CrtYd) (width 0.05))
     (fp_line (start 7.79 -19.71) (end -2.71 -19.71) (layer F.CrtYd) (width 0.05))
+    (fp_text user %R (at 2.54 -20.58) (layer F.Fab)
+      (effects (font (size 1 1) (thickness 0.15)))
+    )
     (pad 3 thru_hole oval (at 5.08 0) (size 1.905 2) (drill 1.1) (layers *.Cu *.Mask)
       (net 14 /DCDC_Fused))
@@
     (effects (font (size 1.2 1.2) (thickness 0.18)))
   )
-  (gr_text "G.Spearing\nLVPDU\n21.038" (at 231.14 83.312) (layer F.SilkS)
-    (effects (font (size 1.2 1.2) (thickness 0.18)))
-  )
+  (gr_text "G.Spearing\nLVPDU\n21.038" (at 233.68 84.455) (layer F.SilkS)
+    (effects (font (size 1.2 1.2) (thickness 0.18)))
+  )
