File: 60V_Indicator/60V_IND/60V_IND.sch (KiCad schematic (older format))
At the start: 6 parts, among them J1 Conn_01x01, J2 Conn_01x01

Commit message: notes from design review 1
Other:
- note added: "HV+\n"
- note added: "HV-\n"
- note added: "TODO: \nChange out three resistors \nfor 1 power resistor\n\nBoard Layout"
Changed lines of the file:
@@
 	1    0    0    -1
 $EndComp
+Text Notes 2975 1725 0    50   ~ 0
+HV+\n
+Text Notes 3000 4025 0    50   ~ 0
+HV-\n
+Text Notes 2600 4750 0    50   ~ 0
+TODO: \nChange out three resistors \nfor 1 power resistor\n\nBoard Layout
 $EndSCHEMATC
