File: HVPDU/HVPDU/HVPDU.kicad_pcb (KiCad board)
At the start: 2 copper layers, 28 parts, among them J1 TE_Connector, J2 TE_Connector, J3 DF22, J4 DF22, J5 Conn_01x14, J6 Conn_01x05, J7 Conn_01x05, Q1 040N03LG, Q2 040N03LG, U1 Vicor_AERO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

Commit message: start layout
Parts:
- removed H7, H8: M3, MountingHole:MountingHole_3.2mm_M3
- added C4: 330uF 25V, AERO_CUSTOM:CAP_18x25_NICH, F.Cu at (206.4, 32.4)
- added C5: 330uF 25V, AERO_CUSTOM:CAP_18x25_NICH, F.Cu at (206.4, 45.7)
- added C6: 47uF 25V, AERO_CUSTOM:CAP_18x25_NICH, F.Cu at (226.7, 32.4)
- added C7: 0.1uF 50v, Capacitor_THT:C_Radial_D10.0mm_H12.5mm_P5.00mm, F.Cu at (226.7, 48.3)
- added D1: LED, LED_SMD:LED_0603_1608Metric_Pad1.05x0.95mm_HandSolder, F.Cu at (104.9, 44.6)
- added R10: R, Resistor_SMD:R_0603_1608Metric_Pad0.98x0.95mm_HandSolder, F.Cu at (109.3, 44.6)
- added R11: R, Resistor_SMD:R_0603_1608Metric_Pad0.98x0.95mm_HandSolder, F.Cu at (113.6, 44.6)
- added R9: 1.0, Resistor_SMD:R_2512_6332Metric_Pad1.40x3.35mm_HandSolder, F.Cu at (187.3, 83.2)
- added RV1: R_POT_TRIM, Potentiometer_THT:Potentiometer_ACP_CA9-V10_Vertical, F.Cu at (103.7, 38.1)
- C1, C2, C3: footprint Capacitor_SMD:C_0603_1608Metric_Pad1.05x0.95mm_HandSolder -> Capacitor_SMD:C_0603_1608Metric_Pad1.08x0.95mm_HandSolder
- F1: footprint AERO-footprints:Fuseholder_Cylinder-5x20mm_Schurter_0031_8201_Horizontal_Open_3d -> AERO_CUSTOM:Fuseholder_Cylinder-5x20mm_Schurter_0031_8201_Horizontal_Open_3d
- J5: footprint AERO-footprints:TE_1-776262-1_14pin_Vertical -> AERO_CUSTOM:TE_1-776262-1_14pin_Vertical; moved to B.Cu
- R2: footprint Resistor_SMD:R_0603_1608Metric_Pad1.05x0.95mm_HandSolder -> Resistor_SMD:R_0603_1608Metric_Pad0.98x0.95mm_HandSolder; moved to B.Cu
- R3, R4, R5: footprint Resistor_SMD:R_0603_1608Metric_Pad1.05x0.95mm_HandSolder -> Resistor_SMD:R_0603_1608Metric_Pad0.98x0.95mm_HandSolder
- R6: footprint Resistor_SMD:R_2512_6332Metric_Pad1.52x3.35mm_HandSolder -> Resistor_SMD:R_2512_6332Metric_Pad1.40x3.35mm_HandSolder
- U1: footprint AERO-footprints:vicor-socket-no-cutouts -> AERO_CUSTOM:vicor-socket
- U3: moved to B.Cu
- moved J2 147.7 mm to (111.1, 54.6), turned to 0 degrees
- moved J1 138.6 mm to (108.0, 20.3)
- moved U1 106.7 mm to (123.8, 29.8)
- moved H5 99.7 mm to (124.5, 116.2)
- moved F1 94.1 mm to (69.8, 47.0), turned to 90 degrees
- moved R7 91.7 mm to (83.8, 76.2), turned to 90 degrees
- moved R8 87.4 mm to (99.7, 114.3), turned to 90 degrees
- moved C1 85.3 mm to (166.4, 76.2)
- moved C3 83.2 mm to (158.8, 79.4), turned to 270 degrees
- moved R3 81.1 mm to (162.6, 76.2)
- moved C2 78.3 mm to (162.6, 88.3), turned to 180 degrees
- moved R1 78.0 mm to (69.8, 86.4), turned to 90 degrees
- moved J4 76.2 mm to (84.5, 114.3)
- moved U2 73.1 mm to (164.5, 82.5), turned to 90 degrees
- moved R4 71.9 mm to (158.8, 83.2), turned to 270 degrees
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Connections:
- J1 pad 2: /IMD_TSV+ -> /TSV+
- J1 pad 3: /SPARE -> /TSV+
- J2 pad 2: /IMD_TSV- -> /TSV-
- J2 pad 3: /SPARE -> /TSV-
- Q2 pad 2: /RED_ON_GND -> Net-(Q2-Pad2)
- U1 pad 2: Net-(U1-Pad2) -> /TR
- U1 pad 3: Net-(U1-Pad3) -> (no net)
- U1 pad 4: Net-(U1-Pad4) -> /FT
Other:
- board outline added: 3.8 x 17.8 mm
- rule pad_to_mask_clearance: 0.051 -> 0
- board text added: "Current Sensor"
- board text added: "GLV"
- board text added: "GND 12 Fault GND 2 GND 3"
- board text added: "GND IN 3 IN 2 IN 1 +5V"
- board text added: "HVPDU BIG DCDC"
- board text added: "IMD"
- board text added: "TMSP -"
- board text added: "TSMP +"
- board text added: "TSV"
- board text added: "TSV+"
- board text added: "TSV-"

Commit message: Change HV PCB Layout
Routing:
- net VCC: track 0.00 -> 50.9 mm, vias 0 -> 2
- net /TSV-: track 0.00 -> 34.2 mm
- net Net-(Q1-Pad2): track 0.00 -> 28.5 mm
- net /TSV+: track 0.00 -> 28.1 mm
- net Net-(Q2-Pad2): track 0.00 -> 18.1 mm
- net /TSAL_on_HVPDU/pass: track 0.00 -> 14.2 mm
- net Net-(R3-Pad2): track 0.00 -> 10.6 mm
- net Net-(Q1-Pad1): track 0.00 -> 5.23 mm
- net Net-(C1-Pad1): track 0.00 -> 4.23 mm
- net /TSAL_on_HVPDU/555_OUT: track 0.00 -> 3.39 mm
