File: HVPDU/HV_DCDC/HV_DCDC.sch (KiCad schematic (older format))
At the start: 18 parts, among them J1 TE_Connector, J2 TE_Connector, J3 DF22, J4 DF22, J5 Conn_01x14, J6 Conn_01x05, J7 Conn_01x05, U1 EPM1510SJ

Commit message: Change HV PCB Layout
Parts:
- U1: symbol AERO_custom_symbols:EPM1510SJ -> HV_DCDC-rescue:EPM1510SJ-AERO_custom_symbols
Changed lines of the file:
@@
 This is an HV board using\nthe EPM1510SJ DCDC \n\nNot used for GLV Charging
 $Comp
-L AERO_custom_symbols:EPM1510SJ U1
+L HV_DCDC-rescue:EPM1510SJ-AERO_custom_symbols U1
 U 1 1 6042841A
 P 2575 1525
