File: HVPDU/HV_DCDC/HV_DCDC.kicad_pcb (KiCad board)
At the start: 2 copper layers, 134.6 x 96.5 mm, 35 parts, among them J1 TE_Connector, J2 TE_Connector, J3 DF22, J4 DF22, J5 Conn_01x14, J6 Conn_01x05, J7 Conn_01x05, Q1 040N03LG, Q2 040N03LG, U1 EPM1510SJ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

Commit message: update layout, finalize
Routing:
- net /+DCDC_OUT: track 139.1 -> 128.8 mm
